Commit message: new xacro

File: urdf/compiled/fr3_link5.urdf (robot description, URDF)
Before this commit: robot fr3, 14 links, 13 joints
Links:
- added link link5_sensor_0; collision sphere radius=0.005; visual sphere radius=0.005
- added link link5_sensor_1; collision sphere radius=0.005; visual sphere radius=0.005
- added link link5_sensor_2; collision sphere radius=0.005; visual sphere radius=0.005
- added link link5_sensor_3; collision sphere radius=0.005; visual sphere radius=0.005
- added link link5_sensor_4; collision sphere radius=0.005; visual sphere radius=0.005
- added link link5_sensor_5; collision sphere radius=0.005; visual sphere radius=0.005
- added link link5_sensor_6; collision sphere radius=0.005; visual sphere radius=0.005
- added link link5_skin; visual mesh filename=package://gentact_ros_tools/meshes/skin/link5.stl scale=1 1 1
Joints:
- added joint link5_base_joint: type fixed, parent fr3_link5, child link5_skin, origin xyz=0 0 0 rpy=0 0 0
- added joint link5_sensor_0_joint: type fixed, parent link5/base_link, child link5_sensor_0, origin xyz=-0.032 -0.092 0.057 rpy=0.488 0.000 -1.431, axis -0.465 -0.066 0.883
- added joint link5_sensor_1_joint: type fixed, parent link5/base_link, child link5_sensor_1, origin xyz=-0.007 -0.131 0.048 rpy=0.848 0.000 -0.160, axis -0.12 -0.74 0.661
- added joint link5_sensor_2_joint: type fixed, parent link5/base_link, child link5_sensor_2, origin xyz=0.023 -0.086 0.060 rpy=0.280 -0.000 1.591, axis 0.276 0.006 0.961
- added joint link5_sensor_3_joint: type fixed, parent link5/base_link, child link5_sensor_3, origin xyz=-0.002 -0.034 0.059 rpy=0.023 0.000 -1.950, axis -0.021 0.008 1.0
- added joint link5_sensor_4_joint: type fixed, parent link5/base_link, child link5_sensor_4, origin xyz=-0.020 0.060 0.059 rpy=0.339 -0.000 -1.569, axis -0.333 -0.001 0.943
- added joint link5_sensor_5_joint: type fixed, parent link5/base_link, child link5_sensor_5, origin xyz=0.049 -0.115 0.025 rpy=1.334 0.000 1.053, axis 0.845 -0.481 0.235
- added joint link5_sensor_6_joint: type fixed, parent link5/base_link, child link5_sensor_6, origin xyz=-0.049 -0.116 0.023 rpy=1.323 0.000 -1.059, axis -0.845 -0.475 0.246

File: urdf/skin/link5.xacro (robot description, xacro)
@@ -1,108 +1,109 @@
 <?xml version="1.0"?>
-<robot name="link5" xmlns:xacro="http://ros.org/wiki/xacro">
-  <!-- Properties -->
-  <xacro:property name="namespace" value="$(arg namespace)" />
-  <xacro:property name="parent" value="$(arg parent)" />
-  <xacro:property name="use_mesh_file" value="true" />
-  <xacro:property name="mesh_file" value="package://gentact_ros_tools/meshes/skin/link5.stl" />
-  <xacro:property name="mass" value="0.3" /> <!-- [kg] -->
-  <xacro:property name="body_width" value="0.3" /> <!-- [m] -->
-  <xacro:property name="body_height" value="0.1" /> <!-- [m] -->
-  <xacro:property name="sensor_length" value="0.05" /> <!-- [m] -->
-  <xacro:property name="sensor_radius" value="0.005" /> <!-- [m] -->
-  <!-- Included URDF Files -->
-  <xacro:include filename="$(find gentact_ros_tools)/urdf/skin/self-cap-base.xacro" />
-  <!-- Instantiate dermis once -->
-  <xacro:dermis_base_macro
-    robot_namespace="${namespace}"
-    parent="${parent}"
-    mass="${mass}"
-    body_width="${body_width}"
-    body_height="${body_height}"
-    use_mesh_file="${use_mesh_file}"
-    mesh_file="${mesh_file}">
-    <inertial>
-      <mass value="${mass}" />
-      <origin xyz="0 0 0" rpy="0 0 0" />
-      <inertia ixx="0.001" ixy="0.0" ixz="0.0" iyy="0.001" iyz="0.0" izz="0.001" />
-    </inertial>
-  </xacro:dermis_base_macro>
-  <!-- Instantiate sensors -->
-  <xacro:self_cap_sensor
-    robot_namespace="${namespace}"
-    parent="${namespace}/base_link"
-    sensor_number="0"
-    sensor_radius="${sensor_radius}"
-    sensor_length="0.057"
-    normal_x="-0.465"
-    normal_y="-0.066"
-    normal_z="0.883">
-    <origin xyz="-0.032 -0.092 0.057" rpy="0.488 0.000 -1.431" />
-  </xacro:self_cap_sensor>
-  <xacro:self_cap_sensor
-    robot_namespace="${namespace}"
-    parent="${namespace}/base_link"
-    sensor_number="1"
-    sensor_radius="${sensor_radius}"
-    sensor_length="0.048"
-    normal_x="-0.120"
-    normal_y="-0.740"
-    normal_z="0.661">
-    <origin xyz="-0.007 -0.131 0.048" rpy="0.848 0.000 -0.160" />
-  </xacro:self_cap_sensor>
-  <xacro:self_cap_sensor
-    robot_namespace="${namespace}"
-    parent="${namespace}/base_link"
-    sensor_number="2"
-    sensor_radius="${sensor_radius}"
-    sensor_length="0.060"
-    normal_x="0.276"
-    normal_y="0.006"
-    normal_z="0.961">
-    <origin xyz="0.023 -0.086 0.060" rpy="0.280 -0.000 1.591" />
-  </xacro:self_cap_sensor>
-  <xacro:self_cap_sensor
-    robot_namespace="${namespace}"
-    parent="${namespace}/base_link"
-    sensor_number="3"
-    sensor_radius="${sensor_radius}"
-    sensor_length="0.059"
-    normal_x="-0.021"
-    normal_y="0.008"
-    normal_z="1.000">
-    <origin xyz="-0.002 -0.034 0.059" rpy="0.023 0.000 -1.950" />
-  </xacro:self_cap_sensor>
-  <xacro:self_cap_sensor
-    robot_namespace="${namespace}"
-    parent="${namespace}/base_link"
-    sensor_number="4"
-    sensor_radius="${sensor_radius}"
-    sensor_length="0.059"
-    normal_x="-0.333"
-    normal_y="-0.001"
-    normal_z="0.943">
-    <origin xyz="-0.020 0.060 0.059" rpy="0.339 -0.000 -1.569" />
-  </xacro:self_cap_sensor>
-  <xacro:self_cap_sensor
-    robot_namespace="${namespace}"
-    parent="${namespace}/base_link"
-    sensor_number="5"
-    sensor_radius="${sensor_radius}"
-    sensor_length="0.025"
-    normal_x="0.845"
-    normal_y="-0.481"
-    normal_z="0.235">
-    <origin xyz="0.049 -0.115 0.025" rpy="1.334 0.000 1.053" />
-  </xacro:self_cap_sensor>
-  <xacro:self_cap_sensor
-    robot_namespace="${namespace}"
-    parent="${namespace}/base_link"
-    sensor_number="6"
-    sensor_radius="${sensor_radius}"
-    sensor_length="0.023"
-    normal_x="-0.845"
-    normal_y="-0.475"
-    normal_z="0.246">
-    <origin xyz="-0.049 -0.116 0.023" rpy="1.323 0.000 -1.059" />
-  </xacro:self_cap_sensor>
+<robot xmlns:xacro="http://ros.org/wiki/xacro">
+  <!-- Macro definition for link5 skin -->
+  <xacro:macro name="link5_skin" params="parent namespace">
+    <!-- Properties -->
+    <xacro:property name="use_mesh_file" value="true" />
+    <xacro:property name="mesh_file" value="package://gentact_ros_tools/meshes/skin/link5.stl" />
+    <xacro:property name="mass" value="0.3" /> <!-- [kg] -->
+    <xacro:property name="body_width" value="0.3" /> <!-- [m] -->
+    <xacro:property name="body_height" value="0.1" /> <!-- [m] -->
+    <xacro:property name="sensor_length" value="0.05" /> <!-- [m] -->
+    <xacro:property name="sensor_radius" value="0.005" /> <!-- [m] -->
+    <!-- Included URDF Files -->
+    <xacro:include filename="$(find gentact_ros_tools)/urdf/skin/self-cap-base.xacro" />
+    <!-- Instantiate dermis once -->
+    <xacro:dermis_base_macro
+      robot_namespace="${namespace}"
+      parent="${parent}"
+      mass="${mass}"
+      body_width="${body_width}"
+      body_height="${body_height}"
+      use_mesh_file="${use_mesh_file}"
+      mesh_file="${mesh_file}">
+      <inertial>
+        <mass value="${mass}" />
+        <origin xyz="0 0 0" rpy="0 0 0" />
+        <inertia ixx="0.001" ixy="0.0" ixz="0.0" iyy="0.001" iyz="0.0" izz="0.001" />
+      </inertial>
+    </xacro:dermis_base_macro>
+    <!-- Instantiate sensors -->
+    <xacro:self_cap_sensor
+      robot_namespace="${namespace}"
+      parent="${namespace}/base_link"
+      sensor_number="0"
+      sensor_radius="${sensor_radius}"
+      sensor_length="0.057"
+      normal_x="-0.465"
+      normal_y="-0.066"
+      normal_z="0.883">
+      <origin xyz="-0.032 -0.092 0.057" rpy="0.488 0.000 -1.431" />
+    </xacro:self_cap_sensor>
+    <xacro:self_cap_sensor
+      robot_namespace="${namespace}"
+      parent="${namespace}/base_link"
+      sensor_number="1"
+      sensor_radius="${sensor_radius}"
+      sensor_length="0.048"
+      normal_x="-0.120"
+      normal_y="-0.740"
+      normal_z="0.661">
+      <origin xyz="-0.007 -0.131 0.048" rpy="0.848 0.000 -0.160" />
+    </xacro:self_cap_sensor>
+    <xacro:self_cap_sensor
+      robot_namespace="${namespace}"
+      parent="${namespace}/base_link"
+      sensor_number="2"
+      sensor_radius="${sensor_radius}"
+      sensor_length="0.060"
+      normal_x="0.276"
+      normal_y="0.006"
+      normal_z="0.961">
+      <origin xyz="0.023 -0.086 0.060" rpy="0.280 -0.000 1.591" />
+    </xacro:self_cap_sensor>
+    <xacro:self_cap_sensor
+      robot_namespace="${namespace}"
+      parent="${namespace}/base_link"
+      sensor_number="3"
+      sensor_radius="${sensor_radius}"
+      sensor_length="0.059"
+      normal_x="-0.021"
+      normal_y="0.008"
+      normal_z="1.000">
+      <origin xyz="-0.002 -0.034 0.059" rpy="0.023 0.000 -1.950" />
+    </xacro:self_cap_sensor>
+    <xacro:self_cap_sensor
+      robot_namespace="${namespace}"
+      parent="${namespace}/base_link"
+      sensor_number="4"
+      sensor_radius="${sensor_radius}"
+      sensor_length="0.059"
+      normal_x="-0.333"
+      normal_y="-0.001"
+      normal_z="0.943">
+      <origin xyz="-0.020 0.060 0.059" rpy="0.339 -0.000 -1.569" />
+    </xacro:self_cap_sensor>
+    <xacro:self_cap_sensor
+      robot_namespace="${namespace}"
+      parent="${namespace}/base_link"
+      sensor_number="5"
+      sensor_radius="${sensor_radius}"
+      sensor_length="0.025"
+      normal_x="0.845"
+      normal_y="-0.481"
+      normal_z="0.235">
+      <origin xyz="0.049 -0.115 0.025" rpy="1.334 0.000 1.053" />
+    </xacro:self_cap_sensor>
+    <xacro:self_cap_sensor
+      robot_namespace="${namespace}"
+      parent="${namespace}/base_link"
+      sensor_number="6"
+      sensor_radius="${sensor_radius}"
+      sensor_length="0.023"
+      normal_x="-0.845"
+      normal_y="-0.475"
+      normal_z="0.246">
+      <origin xyz="-0.049 -0.116 0.023" rpy="1.323 0.000 -1.059" />
+    </xacro:self_cap_sensor>
+  </xacro:macro>
 </robot>

File: urdf/skin/link6.xacro (robot description, xacro)
@@ -1,117 +1,120 @@
 <?xml version="1.0"?>
 <robot name="link6" xmlns:xacro="http://ros.org/wiki/xacro">
-  <!-- Properties -->
-  <xacro:property name="namespace" value="$(arg namespace)" />
-  <xacro:property name="use_mesh_file" value="true" />
-  <xacro:property name="mesh_file" value="package://gentact_ros_tools/meshes/skin/link6.stl" />
-  <xacro:property name="mass" value="0.3" /> <!-- [kg] -->
-  <xacro:property name="body_width" value="0.3" /> <!-- [m] -->
-  <xacro:property name="body_height" value="0.1" /> <!-- [m] -->
-  <xacro:property name="sensor_length" value="0.05" /> <!-- [m] -->
-  <xacro:property name="sensor_radius" value="0.005" /> <!-- [m] -->
-  <!-- Included URDF Files -->
-  <xacro:include filename="$(find gentact_ros_tools)/urdf/skin/self-cap-base.xacro" />
-  <!-- Instantiate dermis once -->
-  <xacro:dermis_base_macro
-    robot_namespace="${namespace}"
-    mass="${mass}"
-    body_width="${body_width}"
-    body_height="${body_height}"
-    use_mesh_file="${use_mesh_file}"
-    mesh_file="${mesh_file}">
-    <inertial>
-      <mass value="${mass}" />
-      <origin xyz="0 0 0" rpy="0 0 0" />
-      <inertia ixx="0.001" ixy="0.0" ixz="0.0" iyy="0.001" iyz="0.0" izz="0.001" />
-    </inertial>
-  </xacro:dermis_base_macro>
-  <!-- Instantiate sensors -->
-  <xacro:self_cap_sensor
-    robot_namespace="${namespace}"
-    parent="${namespace}_skin"
-    sensor_number="0"
-    sensor_radius="0.0"
-    sensor_length="0.057"
-    normal_x="0.474"
-    normal_y="-0.881"
-    normal_z="-0.011">
-    <origin xyz="0.117 -0.045 -0.004" rpy="1.582 0.000 0.494" />
-  </xacro:self_cap_sensor>
-  <xacro:self_cap_sensor
-    robot_namespace="${namespace}"
-    parent="${namespace}_skin"
-    sensor_number="1"
-    sensor_radius="0.0"
-    sensor_length="0.048"
-    normal_x="0.885"
-    normal_y="-0.449"
-    normal_z="0.120">
-    <origin xyz="0.133 -0.025 0.039" rpy="1.451 0.000 1.101" />
-  </xacro:self_cap_sensor>
-  <xacro:self_cap_sensor
-    robot_namespace="${namespace}"
-    parent="${namespace}_skin"
-    sensor_number="2"
-    sensor_radius="0.0"
-    sensor_length="0.060"
-    normal_x="0.991"
-    normal_y="-0.106"
-    normal_z="0.084">
-    <origin xyz="0.140 -0.002 0.030" rpy="1.487 -0.000 1.464" />
-  </xacro:self_cap_sensor>
-  <xacro:self_cap_sensor
-    robot_namespace="${namespace}"
-    parent="${namespace}_skin"
-    sensor_number="3"
-    sensor_radius="0.0"
-    sensor_length="0.059"
-    normal_x="0.477"
-    normal_y="0.879"
-    normal_z="-0.015">
-    <origin xyz="0.113 0.047 0.002" rpy="1.585 -0.000 2.644" />
-  </xacro:self_cap_sensor>
-  <xacro:self_cap_sensor
-    robot_namespace="${namespace}"
-    parent="${namespace}_skin"
-    sensor_number="4"
-    sensor_radius="0.0"
-    sensor_length="0.059"
-    normal_x="0.888"
-    normal_y="0.459"
-    normal_z="0.037">
-    <origin xyz="0.132 0.029 0.018" rpy="1.533 -0.000 2.048" />
-  </xacro:self_cap_sensor>
-  <xacro:self_cap_sensor
-    robot_namespace="${namespace}"
-    parent="${namespace}_skin"
-    sensor_number="5"
-    sensor_radius="0.0"
-    sensor_length="0.025"
-    normal_x="0.995"
-    normal_y="-0.100"
-    normal_z="-0.010">
-    <origin xyz="0.141 -0.001 -0.002" rpy="1.581 -0.000 1.470" />
-  </xacro:self_cap_sensor>
-  <xacro:self_cap_sensor
-    robot_namespace="${namespace}"
-    parent="${namespace}_skin"
-    sensor_number="6"
-    sensor_radius="0.0"
-    sensor_length="0.023"
-    normal_x="0.776"
-    normal_y="-0.631"
-    normal_z="0.030">
-    <origin xyz="0.130 -0.033 0.015" rpy="1.541 -0.000 0.888" />
-  </xacro:self_cap_sensor>
-  <xacro:self_cap_sensor
-    robot_namespace="${namespace}"
-    parent="${namespace}_skin"
-    sensor_number="7"
-    sensor_radius="0.0"
-    sensor_length="0.023"
-    normal_x="-0.092"
-    normal_y="0.992"
-    normal_z="0.083">
-    <origin xyz="0.087 0.051 0.036" rpy="1.488 0.000 -3.049" />
-  </xacro:self_cap_sensor>
+  <!-- Macro definition for link6 skin -->
+  <xacro:macro name="link6_skin" params="parent namespace">
+    <!-- Properties -->
+    <xacro:property name="use_mesh_file" value="true" />
+    <xacro:property name="mesh_file" value="package://gentact_ros_tools/meshes/skin/link6.stl" />
+    <xacro:property name="mass" value="0.3" /> <!-- [kg] -->
+    <xacro:property name="body_width" value="0.3" /> <!-- [m] -->
+    <xacro:property name="body_height" value="0.1" /> <!-- [m] -->
+    <xacro:property name="sensor_length" value="0.05" /> <!-- [m] -->
+    <xacro:property name="sensor_radius" value="0.005" /> <!-- [m] -->
+    <!-- Included URDF Files -->
+    <xacro:include filename="$(find gentact_ros_tools)/urdf/skin/self-cap-base.xacro" />
+    <!-- Instantiate dermis once -->
+    <xacro:dermis_base_macro
+      robot_namespace="${namespace}"
+      parent="${parent}"
+      mass="${mass}"
+      body_width="${body_width}"
+      body_height="${body_height}"
+      use_mesh_file="${use_mesh_file}"
+      mesh_file="${mesh_file}">
+      <inertial>
+        <mass value="${mass}" />
+        <origin xyz="0 0 0" rpy="0 0 0" />
+        <inertia ixx="0.001" ixy="0.0" ixz="0.0" iyy="0.001" iyz="0.0" izz="0.001" />
+      </inertial>
+    </xacro:dermis_base_macro>
+    <!-- Instantiate sensors -->
+    <xacro:self_cap_sensor
+      robot_namespace="${namespace}"
+      parent="${namespace}_skin"
+      sensor_number="0"
+      sensor_radius="0.0"
+      sensor_length="0.057"
+      normal_x="0.474"
+      normal_y="-0.881"
+      normal_z="-0.011">
+      <origin xyz="0.117 -0.045 -0.004" rpy="1.582 0.000 0.494" />
+    </xacro:self_cap_sensor>
+    <xacro:self_cap_sensor
+      robot_namespace="${namespace}"
+      parent="${namespace}_skin"
+      sensor_number="1"
+      sensor_radius="0.0"
+      sensor_length="0.048"
+      normal_x="0.885"
+      normal_y="-0.449"
+      normal_z="0.120">
+      <origin xyz="0.133 -0.025 0.039" rpy="1.451 0.000 1.101" />
+    </xacro:self_cap_sensor>
+    <xacro:self_cap_sensor
+      robot_namespace="${namespace}"
+      parent="${namespace}_skin"
+      sensor_number="2"
+      sensor_radius="0.0"
+      sensor_length="0.060"
+      normal_x="0.991"
+      normal_y="-0.106"
+      normal_z="0.084">
+      <origin xyz="0.140 -0.002 0.030" rpy="1.487 -0.000 1.464" />
+    </xacro:self_cap_sensor>
+    <xacro:self_cap_sensor
+      robot_namespace="${namespace}"
+      parent="${namespace}_skin"
+      sensor_number="3"
+      sensor_radius="0.0"
+      sensor_length="0.059"
+      normal_x="0.477"
+      normal_y="0.879"
+      normal_z="-0.015">
+      <origin xyz="0.113 0.047 0.002" rpy="1.585 -0.000 2.644" />
+    </xacro:self_cap_sensor>
+    <xacro:self_cap_sensor
+      robot_namespace="${namespace}"
+      parent="${namespace}_skin"
+      sensor_number="4"
+      sensor_radius="0.0"
+      sensor_length="0.059"
+      normal_x="0.888"
+      normal_y="0.459"
+      normal_z="0.037">
+      <origin xyz="0.132 0.029 0.018" rpy="1.533 -0.000 2.048" />
+    </xacro:self_cap_sensor>
+    <xacro:self_cap_sensor
+      robot_namespace="${namespace}"
+      parent="${namespace}_skin"
+      sensor_number="5"
+      sensor_radius="0.0"
+      sensor_length="0.025"
+      normal_x="0.995"
+      normal_y="-0.100"
+      normal_z="-0.010">
+      <origin xyz="0.141 -0.001 -0.002" rpy="1.581 -0.000 1.470" />
+    </xacro:self_cap_sensor>
+    <xacro:self_cap_sensor
+      robot_namespace="${namespace}"
+      parent="${namespace}_skin"
+      sensor_number="6"
+      sensor_radius="0.0"
+      sensor_length="0.023"
+      normal_x="0.776"
+      normal_y="-0.631"
+      normal_z="0.030">
+      <origin xyz="0.130 -0.033 0.015" rpy="1.541 -0.000 0.888" />
+    </xacro:self_cap_sensor>
+    <xacro:self_cap_sensor
+      robot_namespace="${namespace}"
+      parent="${namespace}_skin"
+      sensor_number="7"
+      sensor_radius="0.0"
+      sensor_length="0.023"
+      normal_x="-0.092"
+      normal_y="0.992"
+      normal_z="0.083">
+      <origin xyz="0.087 0.051 0.036" rpy="1.488 0.000 -3.049" />
+    </xacro:self_cap_sensor>
+  </xacro:macro>
 </robot>
