Commit message: add all changed for working system before os update

File: urdf/compiled/fr3_12356.urdf (robot description, URDF)
Before this commit: robot fr3, 53 links, 52 joints
Links:
- removed link end_effector
- removed link end_effector_tip
- link link6_skin: geometry visual mesh filename=package://gentact_ros_tools/meshes/skin/self-cap/link6_fanc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 scale=1 1 1
Joints:
- removed joint end_effector_joint
- removed joint end_effector_tip_joint
- joint link3_sensor_0_joint: axis -0.71 -0.691 0.137 -> -0.059 0.982 0.178; origin xyz=-0.041 -0.037 -0.071 rpy=1.433 0.000 -0.799 -> xyz=0.008 0.051 -0.043 rpy=1.392 0.000 -3.082
- joint link3_sensor_1_joint: axis -0.878 0.457 0.145 -> 0.217 0.956 -0.196; origin xyz=-0.050 0.023 -0.063 rpy=1.426 0.000 -2.050 -> xyz=0.097 0.113 -0.015 rpy=1.768 -0.000 2.918
- joint link3_sensor_2_joint: axis 0.056 0.301 -0.952 -> -0.71 -0.691 0.137; origin xyz=0.085 0.086 -0.050 rpy=-0.311 3.142 -0.185 -> xyz=-0.041 -0.037 -0.071 rpy=1.433 0.000 -0.799
- joint link3_sensor_3_joint: axis -0.371 0.89 -0.264 -> 0.386 0.844 0.373; origin xyz=0.057 0.108 -0.019 rpy=1.838 0.000 -2.747 -> xyz=0.107 0.106 0.026 rpy=1.189 -0.000 2.713
- joint link3_sensor_5_joint: axis -0.059 0.982 0.178 -> -0.371 0.89 -0.264; origin xyz=0.008 0.051 -0.043 rpy=1.392 0.000 -3.082 -> xyz=0.057 0.108 -0.019 rpy=1.838 0.000 -2.747
- joint link3_sensor_6_joint: axis 0.217 0.956 -0.196 -> -0.878 0.457 0.145; origin xyz=0.097 0.113 -0.015 rpy=1.768 -0.000 2.918 -> xyz=-0.050 0.023 -0.063 rpy=1.426 0.000 -2.050
- joint link3_sensor_7_joint: axis 0.386 0.844 0.373 -> 0.056 0.301 -0.952; origin xyz=0.107 0.106 0.026 rpy=1.189 -0.000 2.713 -> xyz=0.085 0.086 -0.050 rpy=-0.311 3.142 -0.185

File: urdf/compiled/fr3_2356_fancy.urdf (robot description, URDF)
Before this commit: robot fr3, 44 links, 43 joints
Links:
- removed link end_effector
- removed link end_effector_tip
- link link6_skin: geometry visual mesh filename=package://gentact_ros_tools/meshes/skin/self-cap/link6_fanc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 scale=1 1 1
Joints:
- removed joint end_effector_joint
- removed joint end_effector_tip_joint
- joint link2_base_joint: origin xyz=0 0 0 rpy=0 0 0 -> xyz=0 0 0 rpy=1.5707 0 0
- joint link3_sensor_0_joint: axis -0.71 -0.691 0.137 -> -0.059 0.982 0.178; origin xyz=-0.041 -0.037 -0.071 rpy=1.433 0.000 -0.799 -> xyz=0.008 0.051 -0.043 rpy=1.392 0.000 -3.082
- joint link3_sensor_1_joint: axis -0.878 0.457 0.145 -> 0.217 0.956 -0.196; origin xyz=-0.050 0.023 -0.063 rpy=1.426 0.000 -2.050 -> xyz=0.097 0.113 -0.015 rpy=1.768 -0.000 2.918
- joint link3_sensor_2_joint: axis 0.056 0.301 -0.952 -> -0.71 -0.691 0.137; origin xyz=0.085 0.086 -0.050 rpy=-0.311 3.142 -0.185 -> xyz=-0.041 -0.037 -0.071 rpy=1.433 0.000 -0.799
- joint link3_sensor_3_joint: axis -0.371 0.89 -0.264 -> 0.386 0.844 0.373; origin xyz=0.057 0.108 -0.019 rpy=1.838 0.000 -2.747 -> xyz=0.107 0.106 0.026 rpy=1.189 -0.000 2.713
- joint link3_sensor_5_joint: axis -0.059 0.982 0.178 -> -0.371 0.89 -0.264; origin xyz=0.008 0.051 -0.043 rpy=1.392 0.000 -3.082 -> xyz=0.057 0.108 -0.019 rpy=1.838 0.000 -2.747
- joint link3_sensor_6_joint: axis 0.217 0.956 -0.196 -> -0.878 0.457 0.145; origin xyz=0.097 0.113 -0.015 rpy=1.768 -0.000 2.918 -> xyz=-0.050 0.023 -0.063 rpy=1.426 0.000 -2.050
- joint link3_sensor_7_joint: axis 0.386 0.844 0.373 -> 0.056 0.301 -0.952; origin xyz=0.107 0.106 0.026 rpy=1.189 -0.000 2.713 -> xyz=0.085 0.086 -0.050 rpy=-0.311 3.142 -0.185

File: urdf/compiled/fr3_56_fancy.urdf (robot description, URDF)
Before this commit: robot fr3, 31 links, 30 joints
Links:
- removed link fr3_hand
- removed link fr3_hand_tcp
- removed link fr3_leftfinger
- removed link fr3_link8
- removed link fr3_rightfinger
- removed link link5_sensor_6
- link link5_sensor_0: geometry collision sphere radius=0.0; visual sphere radius=0.0
- link link5_sensor_1: geometry collision sphere radius=0.0; visual sphere radius=0.0
- link link5_sensor_2: geometry collision sphere radius=0.0; visual sphere radius=0.0
- link link5_sensor_3: geometry collision sphere radius=0.0; visual sphere radius=0.0
- link link5_sensor_4: geometry collision sphere radius=0.0; visual sphere radius=0.0
- link link5_sensor_5: geometry collision sphere radius=0.0; visual sphere radius=0.0
- link link6_skin: geometry visual mesh filename=package://gentact_ros_tools/meshes/skin/self-cap/link6_fanc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 scale=1 1 1
Joints:
- removed joint fr3_finger_joint1
- removed joint fr3_finger_joint2
- removed joint fr3_hand_joint
- removed joint fr3_hand_tcp_joint
- removed joint fr3_joint8
- removed joint link5_sensor_6_joint
- joint link5_sensor_0_joint: axis -0.465 -0.066 0.883 -> -0.018 0.953 -0.304; origin xyz=-0.032 -0.092 0.057 rpy=0.488 0.000 -1.431 -> xyz=-0.000 0.096 -0.184 rpy=-1.262 3.142 0.019; parent link5/base_link -> link5_skin
- joint link5_sensor_1_joint: axis -0.12 -0.74 0.661 -> -0.05 0.941 -0.335; origin xyz=-0.007 -0.131 0.048 rpy=0.848 0.000 -0.160 -> xyz=-0.007 0.127 -0.038 rpy=-1.229 -3.142 0.054; parent link5/base_link -> link5_skin
- joint link5_sensor_2_joint: axis 0.276 0.006 0.961 -> -0.23 0.956 -0.183; origin xyz=0.023 -0.086 0.060 rpy=0.280 -0.000 1.591 -> xyz=-0.016 0.104 -0.138 rpy=1.754 0.000 -2.906; parent link5/base_link -> link5_skin
- joint link5_sensor_3_joint: axis -0.021 0.008 1.0 -> -0.092 0.902 0.422; origin xyz=-0.002 -0.034 0.059 rpy=0.023 0.000 -1.950 -> xyz=-0.007 0.133 0.023 rpy=1.136 0.000 -3.040; parent link5/base_link -> link5_skin
- joint link5_sensor_4_joint: axis -0.333 -0.001 0.943 -> 0.375 0.908 -0.188; origin xyz=-0.020 0.060 0.059 rpy=0.339 -0.000 -1.569 -> xyz=0.026 0.130 -0.013 rpy=1.760 -0.000 2.750; parent link5/base_link -> link5_skin
- joint link5_sensor_5_joint: axis 0.845 -0.481 0.235 -> -0.049 0.985 -0.167; origin xyz=0.049 -0.115 0.025 rpy=1.334 0.000 1.053 -> xyz=-0.004 0.115 -0.089 rpy=-1.403 -3.142 0.049; parent link5/base_link -> link5_skin
- joint link6_base_joint: origin xyz=0 0 0 rpy=0 0 0 -> xyz=0 0 0 rpy=-1.57079632679 0 0

File: urdf/compiled/fr3_link5.urdf (robot description, URDF)
Before this commit: robot fr3, 31 links, 30 joints
Links:
- removed link fr3_hand
- removed link fr3_hand_tcp
- removed link fr3_leftfinger
- removed link fr3_link8
- removed link fr3_rightfinger
- removed link link6_sensor_0
- removed link link6_sensor_1
- removed link link6_sensor_2
- removed link link6_sensor_3
- removed link link6_sensor_4
- removed link link6_sensor_5
- removed link link6_sensor_6
- removed link link6_sensor_7
- removed link link6_skin
- added link link5_sensor_7; collision sphere radius=0.005; visual sphere radius=0.005
- link link5_skin: geometry visual mesh filename=package://gentact_ros_tools/meshes/skin/spad/link5_spad.stl scale=1 1 1
Joints:
- removed joint fr3_finger_joint1
- removed joint fr3_finger_joint2
- removed joint fr3_hand_joint
- removed joint fr3_hand_tcp_joint
- removed joint fr3_joint8
- removed joint link6_base_joint
- removed joint link6_sensor_0_joint
- removed joint link6_sensor_1_joint
- removed joint link6_sensor_2_joint
- removed joint link6_sensor_3_joint
- removed joint link6_sensor_4_joint
- removed joint link6_sensor_5_joint
- removed joint link6_sensor_6_joint
- removed joint link6_sensor_7_joint
- added joint link5_sensor_7_joint: type fixed, parent link5_skin, child link5_sensor_7, origin xyz=-0.019 0.0595 0.054 rpy=-0.002 -0.376 0.0, axis -0.367 0.002 0.93
- joint link5_base_joint: origin xyz=0 0 0 rpy=0 0 0 -> xyz=0 0.06 -0.083 rpy=1.4 3.14 3.14
- joint link5_sensor_0_joint: axis -0.465 -0.066 0.883 -> -0.045 -0.002 0.999; origin xyz=-0.032 -0.092 0.057 rpy=0.488 0.000 -1.431 -> xyz=0.0 -0.0385 0.054 rpy=0.002 -0.045 0.0; parent link5/base_link -> link5_skin
- joint link5_sensor_1_joint: axis -0.12 -0.74 0.661 -> -0.039 0.084 0.996; origin xyz=-0.007 -0.131 0.048 rpy=0.848 0.000 -0.160 -> xyz=-0.002 -0.0795 0.058 rpy=-0.084 -0.039 0.002; parent link5/base_link -> link5_skin
- joint link5_sensor_2_joint: axis 0.276 0.006 0.961 -> -0.045 -0.031 0.998; origin xyz=0.023 -0.086 0.060 rpy=0.280 -0.000 1.591 -> xyz=-0.002 0.0035 0.055 rpy=0.031 -0.045 -0.001; parent link5/base_link -> link5_skin
- joint link5_sensor_3_joint: axis -0.021 0.008 1.0 -> 0.379 -0.002 0.925; origin xyz=-0.002 -0.034 0.059 rpy=0.023 0.000 -1.950 -> xyz=0.023 0.0585 0.052 rpy=0.002 0.389 0.0; parent link5/base_link -> link5_skin
- joint link5_sensor_4_joint: axis -0.333 -0.001 0.943 -> 0.866 -0.368 0.34; origin xyz=-0.020 0.060 0.059 rpy=0.339 -0.000 -1.569 -> xyz=0.047 -0.1075 0.026 rpy=0.825 1.046 0.494; parent link5/base_link -> link5_skin
- joint link5_sensor_5_joint: axis 0.845 -0.481 0.235 -> 0.049 0.408 0.912; origin xyz=0.049 -0.115 0.025 rpy=1.334 0.000 1.053 -> xyz=0.003 0.1235 0.043 rpy=0.421 -0.049 0.01; parent link5/base_link -> link5_skin
- joint link5_sensor_6_joint: axis -0.845 -0.475 0.246 -> -0.097 -0.783 0.615; origin xyz=-0.049 -0.116 0.023 rpy=1.323 0.000 -1.059 -> xyz=-0.004 -0.1295 0.044 rpy=0.905 -0.097 -0.047; parent link5/base_link -> link5_skin

File: urdf/compiled/robot.urdf (robot description, URDF)
Before this commit: robot fr3, 51 links, 50 joints
Links:
- removed link end_effector
- removed link end_effector_tip
- removed link link2_sensor_0
- removed link link2_sensor_1
- removed link link2_sensor_2
- removed link link2_sensor_3
- removed link link2_sensor_4
- removed link link2_sensor_5
- removed link link2_sensor_6
- removed link link2_skin
- removed link link3_sensor_0
- removed link link3_sensor_1
- removed link link3_sensor_2
- removed link link3_sensor_3
- removed link link3_sensor_4
- removed link link3_sensor_5
- removed link link3_sensor_6
- removed link link3_sensor_7
- removed link link3_skin
- removed link link4_sensor_0
- removed link link4_sensor_1
- removed link link4_sensor_2
- removed link link4_sensor_3
- removed link link4_sensor_4
- removed link link4_sensor_5
- removed link link4_skin
- removed link link6_sensor_0
- removed link link6_sensor_1
- removed link link6_sensor_2
- removed link link6_sensor_3
- removed link link6_sensor_4
- removed link link6_sensor_5
- removed link link6_sensor_6
- removed link link6_sensor_7
- removed link link6_skin
- added link link5_sensor_6; collision sphere radius=0.005; visual sphere radius=0.005
- added link link5_sensor_7; collision sphere radius=0.005; visual sphere radius=0.005
- link link5_sensor_0: geometry collision sphere radius=0.005; visual sphere radius=0.005
- link link5_sensor_1: geometry collision sphere radius=0.005; visual sphere radius=0.005
- link link5_sensor_2: geometry collision sphere radius=0.005; visual sphere radius=0.005
- link link5_sensor_3: geometry collision sphere radius=0.005; visual sphere radius=0.005
- link link5_sensor_4: geometry collision sphere radius=0.005; visual sphere radius=0.005
- link link5_sensor_5: geometry collision sphere radius=0.005; visual sphere radius=0.005
- link link5_skin: geometry visual mesh filename=package://gentact_ros_tools/meshes/skin/spad/link5_spad.stl scale=1 1 1
Joints:
- removed joint end_effector_joint
- removed joint end_effector_tip_joint
- removed joint link2_base_joint
- removed joint link2_sensor_0_joint
- removed joint link2_sensor_1_joint
- removed joint link2_sensor_2_joint
- removed joint link2_sensor_3_joint
- removed joint link2_sensor_4_joint
- removed joint link2_sensor_5_joint
- removed joint link2_sensor_6_joint
- removed joint link3_base_joint
- removed joint link3_sensor_0_joint
- removed joint link3_sensor_1_joint
- removed joint link3_sensor_2_joint
- removed joint link3_sensor_3_joint
- removed joint link3_sensor_4_joint
- removed joint link3_sensor_5_joint
- removed joint link3_sensor_6_joint
- removed joint link3_sensor_7_joint
- removed joint link4_base_joint
- removed joint link4_sensor_0_joint
- removed joint link4_sensor_1_joint
- removed joint link4_sensor_2_joint
- removed joint link4_sensor_3_joint
- removed joint link4_sensor_4_joint
- removed joint link4_sensor_5_joint
- removed joint link6_base_joint
- removed joint link6_sensor_0_joint
- removed joint link6_sensor_1_joint
- removed joint link6_sensor_2_joint
- removed joint link6_sensor_3_joint
- removed joint link6_sensor_4_joint
- removed joint link6_sensor_5_joint
- removed joint link6_sensor_6_joint
- removed joint link6_sensor_7_joint
- added joint link5_sensor_6_joint: type fixed, parent link5_skin, child link5_sensor_6, origin xyz=-0.004 -0.1295 0.044 rpy=0.905 -0.097 -0.047, axis -0.097 -0.783 0.615
- added joint link5_sensor_7_joint: type fixed, parent link5_skin, child link5_sensor_7, origin xyz=-0.019 0.0595 0.054 rpy=-0.002 -0.376 0.0, axis -0.367 0.002 0.93
- joint link5_base_joint: origin xyz=0 0 0 rpy=0 0 0 -> xyz=0 0.06 -0.083 rpy=1.4 3.14 3.14
- joint link5_sensor_0_joint: axis -0.018 0.953 -0.304 -> -0.045 -0.002 0.999; origin xyz=-0.000 0.096 -0.184 rpy=-1.262 3.142 0.019 -> xyz=0.0 -0.0385 0.054 rpy=0.002 -0.045 0.0
- joint link5_sensor_1_joint: axis -0.05 0.941 -0.335 -> -0.039 0.084 0.996; origin xyz=-0.007 0.127 -0.038 rpy=-1.229 -3.142 0.054 -> xyz=-0.002 -0.0795 0.058 rpy=-0.084 -0.039 0.002
- joint link5_sensor_2_joint: axis -0.23 0.956 -0.183 -> -0.045 -0.031 0.998; origin xyz=-0.016 0.104 -0.138 rpy=1.754 0.000 -2.906 -> xyz=-0.002 0.0035 0.055 rpy=0.031 -0.045 -0.001
- joint link5_sensor_3_joint: axis -0.092 0.902 0.422 -> 0.379 -0.002 0.925; origin xyz=-0.007 0.133 0.023 rpy=1.136 0.000 -3.040 -> xyz=0.023 0.0585 0.052 rpy=0.002 0.389 0.0
- joint link5_sensor_4_joint: axis 0.375 0.908 -0.188 -> 0.866 -0.368 0.34; origin xyz=0.026 0.130 -0.013 rpy=1.760 -0.000 2.750 -> xyz=0.047 -0.1075 0.026 rpy=0.825 1.046 0.494
- joint link5_sensor_5_joint: axis -0.049 0.985 -0.167 -> 0.049 0.408 0.912; origin xyz=-0.004 0.115 -0.089 rpy=-1.403 -3.142 0.049 -> xyz=0.003 0.1235 0.043 rpy=0.421 -0.049 0.01

File: urdf/skin/link5_spad.xacro (robot description, xacro)
@@ -34,5 +34,5 @@
       normal_y="-0.002"
       normal_z="0.999">
-      <origin xyz="0.0 -0.0385 0.054" rpy="0.002 -0.045 0.0" />
+      <origin xyz="0.0 -0.039 0.054" rpy="0.002 -0.045 0.0" />
     </xacro:self_cap_sensor>
     <xacro:self_cap_sensor
@@ -45,5 +45,5 @@
       normal_y="0.084"
       normal_z="0.996">
-      <origin xyz="-0.002 -0.0795 0.058" rpy="-0.084 -0.039 0.002" />
+      <origin xyz="-0.002 -0.080 0.058" rpy="-0.084 -0.039 0.002" />
     </xacro:self_cap_sensor>
     <xacro:self_cap_sensor
@@ -56,5 +56,5 @@
       normal_y="-0.031"
       normal_z="0.998">
-      <origin xyz="-0.002 0.0035 0.055" rpy="0.031 -0.045 -0.001" />
+      <origin xyz="-0.002 0.003 0.055" rpy="0.031 -0.045 -0.001" />
     </xacro:self_cap_sensor>
     <xacro:self_cap_sensor
@@ -67,5 +67,5 @@
       normal_y="-0.002"
       normal_z="0.925">
-      <origin xyz="0.023 0.0585 0.052" rpy="0.002 0.389 0.0" />
+      <origin xyz="0.023 0.058 0.052" rpy="0.002 0.389 0.0" />
     </xacro:self_cap_sensor>
     <xacro:self_cap_sensor
@@ -78,5 +78,5 @@
       normal_y="-0.368"
       normal_z="0.34">
-      <origin xyz="0.047 -0.1075 0.026" rpy="0.825 1.046 0.494" />
+      <origin xyz="0.047 -0.108 0.026" rpy="0.825 1.046 0.494" />
     </xacro:self_cap_sensor>
     <xacro:self_cap_sensor
@@ -89,5 +89,5 @@
       normal_y="0.408"
       normal_z="0.912">
-      <origin xyz="0.003 0.1235 0.043" rpy="0.421 -0.049 0.01" />
+      <origin xyz="0.003 0.123 0.043" rpy="0.421 -0.049 0.01" />
     </xacro:self_cap_sensor>
     <xacro:self_cap_sensor
@@ -100,5 +100,5 @@
       normal_y="-0.783"
       normal_z="0.615">
-      <origin xyz="-0.004 -0.1295 0.044" rpy="0.905 -0.097 -0.047" />
+      <origin xyz="-0.004 -0.130 0.044" rpy="0.905 -0.097 -0.047" />
     </xacro:self_cap_sensor>
     <xacro:self_cap_sensor
@@ -111,5 +111,5 @@
       normal_y="0.002"
       normal_z="0.93">
-      <origin xyz="-0.019 0.0595 0.054" rpy="-0.002 -0.376 0.0" />
+      <origin xyz="-0.019 0.059 0.054" rpy="-0.002 -0.376 0.0" />
     </xacro:self_cap_sensor>
   </xacro:macro>
