Commit message: broke the robot descr

File: urdf/compiled/fr3_hybrid_skin.urdf (robot description, URDF)
Before this commit: robot fr3, 61 links, 60 joints
Joints:
- joint link5_back_base_joint: parent fr3_link5 -> fr3_link5_back
- joint link5_front_base_joint: parent fr3_link5 -> fr3_link5_front

File: urdf/robot/fr3_full_skin.xacro (robot description, xacro)
@@ -208,5 +208,5 @@
   <xacro:if value="${link5_front_skin_value != ''}">
     <xacro:include filename="$(arg link5_front_skin)" />
-    <xacro:link5_front_skin parent="fr3_link5" namespace="link5" />
+    <xacro:link5_front_skin parent="fr3_link5_front" namespace="link5_front" />
   </xacro:if>
   <!-- Include the skin for link5 if specified -->
@@ -214,5 +214,5 @@
   <xacro:if value="${link5_back_skin_value != ''}">
     <xacro:include filename="$(arg link5_back_skin)" />
-    <xacro:link5_back_skin parent="fr3_link5" namespace="link5" />
+    <xacro:link5_back_skin parent="fr3_link5_back" namespace="link5_back" />
   </xacro:if>
   <!-- sub-link defining detailed meshes for collision with environment -->

Commit message: resolved the robot description error by removing _front and _back from link5 parent=link5 shenanigans

File: urdf/compiled/fr3_hybrid_skin.urdf (robot description, URDF)
Before this commit: robot fr3, 61 links, 60 joints
Joints:
- joint link5_back_base_joint: parent fr3_link5_back -> fr3_link5
- joint link5_front_base_joint: parent fr3_link5_front -> fr3_link5

File: urdf/robot/fr3_full_skin.xacro (robot description, xacro)
@@ -208,5 +208,5 @@
   <xacro:if value="${link5_front_skin_value != ''}">
     <xacro:include filename="$(arg link5_front_skin)" />
-    <xacro:link5_front_skin parent="fr3_link5_front" namespace="link5_front" />
+    <xacro:link5_front_skin parent="fr3_link5" namespace="link5_front" />
   </xacro:if>
   <!-- Include the skin for link5 if specified -->
@@ -214,5 +214,5 @@
   <xacro:if value="${link5_back_skin_value != ''}">
     <xacro:include filename="$(arg link5_back_skin)" />
-    <xacro:link5_back_skin parent="fr3_link5_back" namespace="link5_back" />
+    <xacro:link5_back_skin parent="fr3_link5" namespace="link5_back" />
   </xacro:if>
   <!-- sub-link defining detailed meshes for collision with environment -->

Commit message: fixed link5 front and back skins

File: urdf/compiled/fr3_hybrid_skin.urdf (robot description, URDF)
Before this commit: robot fr3, 61 links, 60 joints
Links:
- removed link link5_back_sensor_4
- removed link link5_back_sensor_5
- added link link5_front_sensor_4
- added link link5_front_sensor_5
Joints:
- removed joint link5_back_sensor_4_joint
- removed joint link5_back_sensor_5_joint
- added joint link5_front_sensor_4_joint: type fixed, parent link5_front_skin, child link5_front_sensor_4, origin xyz=0.049 0.108 0.014 rpy=1.278 0.000 2.016, axis 0.864 0.412 0.289
- added joint link5_front_sensor_5_joint: type fixed, parent link5_front_skin, child link5_front_sensor_5, origin xyz=-0.050 0.106 0.016 rpy=1.282 0.000 -2.017, axis -0.865 0.414 0.285
- joint link3_sensor_0_joint: axis 0 0 0 -> -0.46 0.875 0.151
- joint link3_sensor_1_joint: axis 0 0 0 -> -0.371 0.89 -0.264
- joint link3_sensor_2_joint: axis 0 0 0 -> 0.732 0.662 0.16
- joint link3_sensor_3_joint: axis 0 0 0 -> -0.885 -0.441 0.148
- joint link3_sensor_4_joint: axis 0 0 0 -> -0.689 0.2 0.697
- joint link5_back_sensor_0_joint: axis -0.048 0.984 -0.173 -> -0.366 -0.69 0.625; origin xyz=-0.006 0.114 -0.097 rpy=-1.397 -3.142 0.049 -> xyz=-0.025 -0.042 -0.191 rpy=0.896 0.000 -0.487
- joint link5_back_sensor_1_joint: axis -0.374 0.909 -0.182 -> -0.024 -0.383 0.923; origin xyz=-0.021 0.102 -0.151 rpy=1.754 0.000 -2.751 -> xyz=-0.002 0.022 -0.152 rpy=0.394 0.000 -0.062
- joint link5_back_sensor_2_joint: axis -0.048 0.972 -0.232 -> -0.028 -0.982 0.189; origin xyz=-0.002 0.135 -0.018 rpy=-1.337 3.142 0.049 -> xyz=-0.000 0.058 -0.115 rpy=1.380 -0.000 -0.028
- joint link5_back_sensor_3_joint: axis 0.376 0.908 -0.187 -> 0.377 -0.687 0.621; origin xyz=0.020 0.103 -0.148 rpy=1.758 -0.000 2.749 -> xyz=0.027 -0.041 -0.191 rpy=0.901 -0.000 0.501
- joint link5_front_sensor_0_joint: axis 0 0 0 -> -0.048 0.984 -0.173; origin xyz=-0.025 -0.042 -0.191 rpy=0.896 0.000 -0.487 -> xyz=-0.006 0.114 -0.097 rpy=-1.397 -3.142 0.049
- joint link5_front_sensor_1_joint: axis 0 0 0 -> -0.374 0.909 -0.182; origin xyz=-0.002 0.022 -0.152 rpy=0.394 0.000 -0.062 -> xyz=-0.021 0.102 -0.151 rpy=1.754 0.000 -2.751
- joint link5_front_sensor_2_joint: axis 0 0 0 -> -0.048 0.972 -0.232; origin xyz=-0.000 0.058 -0.115 rpy=1.380 -0.000 -0.028 -> xyz=-0.002 0.135 -0.018 rpy=-1.337 3.142 0.049
- joint link5_front_sensor_3_joint: axis 0 0 0 -> 0.376 0.908 -0.187; origin xyz=0.027 -0.041 -0.191 rpy=0.901 -0.000 0.501 -> xyz=0.020 0.103 -0.148 rpy=1.758 -0.000 2.749
