Commit message: add h1_2 skins

File: urdf/compiled/h1_2_handless_tof.urdf (robot description, URDF)
Before this commit: robot h1_2, 40 links, 39 joints
Links:
- removed link right_shoulder_roll_sensor_6
- added link left_elbow_sensor_0
- added link left_elbow_sensor_1
- added link left_elbow_sensor_2
- added link left_elbow_sensor_3
- added link left_elbow_sensor_4
- added link left_elbow_sensor_5
- added link left_elbow_sensor_6
- added link left_elbow_sensor_7
- added link left_elbow_sensor_8
- added link left_elbow_skin; visual mesh filename=package://gentact_ros_tools_hybrid/meshes/h1_2/skin/tof/elb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 scale=1 1 1
- added link right_shoulder_yaw_sensor_0
- added link right_shoulder_yaw_sensor_1
- added link right_shoulder_yaw_sensor_2
- added link right_shoulder_yaw_sensor_3
- added link right_shoulder_yaw_sensor_4
- added link right_shoulder_yaw_sensor_5
- added link right_shoulder_yaw_skin; visual mesh filename=package://gentact_ros_tools_hybrid/meshes/h1_2/skin/tof/sho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 scale=1 1 1
- link right_shoulder_roll_skin: geometry visual mesh filename=package://gentact_ros_tools_hybrid/meshes/h1_2/skin/tof/sho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 scale=1 1 1
Joints:
- removed joint right_shoulder_roll_sensor_6_joint
- added joint left_elbow_base_joint: type fixed, parent left_elbow_link, child left_elbow_skin, origin xyz=0 0 0 rpy=0 0 0
- added joint left_elbow_sensor_0_joint: type fixed, parent left_elbow_skin, child left_elbow_sensor_0, origin xyz=-0.0054705264046788216 -0.01703549548983574 -0.02506975084543228 rpy=1.6108835935592651 3.0750507695742613e-10 -0.003349356586113572, axis -0.0033466597087681293 -0.9991910457611084 -0.04007663577795029
- added joint left_elbow_sensor_1_joint: type fixed, parent left_elbow_skin, child left_elbow_sensor_1, origin xyz=0.09776215255260468 -0.009773069061338902 -0.003952523693442345 rpy=1.4375799894332886 -2.939074983387968e-09 0.032789308577775955, axis 0.03249296545982361 -0.9906070828437805 0.1328226923942566
- added joint left_elbow_sensor_2_joint: type fixed, parent left_elbow_skin, child left_elbow_sensor_2, origin xyz=0.02981957234442234 -0.015662170946598053 0.0170421302318573 rpy=1.4639254808425903 -1.415918404745753e-08 0.13112856447696686, axis 0.13000711798667908 -0.9857586622238159 0.10666757822036743
- added joint left_elbow_sensor_3_joint: type fixed, parent left_elbow_skin, child left_elbow_sensor_3, origin xyz=0.03183375298976898 -0.012470245361328125 -0.038558200001716614 rpy=2.034855842590332 1.6719945428178562e-09 0.1387859433889389, axis 0.12371029704809189 -0.8856444358825684 -0.4475819766521454
- added joint left_elbow_sensor_4_joint: type fixed, parent left_elbow_skin, child left_elbow_sensor_4, origin xyz=0.09520145505666733 0.008756054565310478 0.02564341574907303 rpy=0.5687653422355652 -1.8162769066520923e-08 0.12151739746332169, axis 0.06528738886117935 -0.5346206426620483 0.8425664901733398
- added joint left_elbow_sensor_5_joint: type fixed, parent left_elbow_skin, child left_elbow_sensor_5, origin xyz=-0.006869952194392681 -0.017091382294893265 0.005429353564977646 rpy=1.5707944631576538 2.0792034760575007e-10 0.004111796617507935, axis 0.004111784510314465 -0.9999915361404419 2.02366391022224e-06
- added joint left_elbow_sensor_6_joint: type fixed, parent left_elbow_skin, child left_elbow_sensor_6, origin xyz=0.08788560330867767 0.03748124837875366 0.03188776969909668 rpy=0.10568315535783768 -2.4437664336574016e-08 3.049027919769287, axis 0.00975038856267929 0.10503476858139038 0.9944207668304443
- added joint left_elbow_sensor_7_joint: type fixed, parent left_elbow_skin, child left_elbow_sensor_7, origin xyz=0.08021856844425201 0.01752631552517414 -0.05247209593653679 rpy=2.8729567527770996 -1.6629815746682652e-08 0.188669815659523, axis 0.049779538065195084 -0.26070669293403625 -0.9641338586807251
- added joint left_elbow_sensor_8_joint: type fixed, parent left_elbow_skin, child left_elbow_sensor_8, origin xyz=0.06785736232995987 -0.006429128348827362 -0.03632089123129845 rpy=2.093989372253418 -2.5215447507775934e-09 0.17718012630939484, axis 0.15267664194107056 -0.8526670932769775 -0.4996485412120819
- added joint right_shoulder_yaw_base_joint: type fixed, parent right_shoulder_yaw_link, child right_shoulder_yaw_skin, origin xyz=0 0 0 rpy=0 0 0
- added joint right_shoulder_yaw_sensor_0_joint: type fixed, parent right_shoulder_yaw_skin, child right_shoulder_yaw_sensor_0, origin xyz=0.04118751734495163 -0.004814512562006712 -0.08737954497337341 rpy=1.8597503900527954 1.1286831025358879e-08 1.4440847635269165, axis 0.9508576989173889 -0.12113388627767563 -0.28494971990585327
- added joint right_shoulder_yaw_sensor_1_joint: type fixed, parent right_shoulder_yaw_skin, child right_shoulder_yaw_sensor_1, origin xyz=-0.035796575248241425 -0.03355425223708153 -0.04064032435417175 rpy=1.646294355392456 1.8119585831755103e-09 -0.7687416672706604, axis -0.6932508945465088 -0.7167385220527649 -0.07542620599269867
- added joint right_shoulder_yaw_sensor_2_joint: type fixed, parent right_shoulder_yaw_skin, child right_shoulder_yaw_sensor_2, origin xyz=0.0068807341158390045 -0.038329385221004486 -0.07258914411067963 rpy=1.8499118089675903 -2.4386073160798105e-09 0.04182104021310806, axis 0.04019082337617874 -0.9604589939117432 -0.2755054235458374
- added joint right_shoulder_yaw_sensor_3_joint: type fixed, parent right_shoulder_yaw_skin, child right_shoulder_yaw_sensor_3, origin xyz=-0.04953809827566147 -0.003564621554687619 -0.0796278566122055 rpy=1.571201205253601 3.790614400145387e-08 -1.4650746583938599, axis -0.9944165349006653 -0.10552489757537842 -0.0004047837865073234
- added joint right_shoulder_yaw_sensor_4_joint: type fixed, parent right_shoulder_yaw_skin, child right_shoulder_yaw_sensor_4, origin xyz=-0.00878828577697277 0.04951019585132599 -0.0318453386425972 rpy=1.5546531677246094 -2.4349319005523284e-08 -3.0059409141540527, axis -0.13521844148635864 0.9906842708587646 0.01614234782755375
- added joint right_shoulder_yaw_sensor_5_joint: type fixed, parent right_shoulder_yaw_skin, child right_shoulder_yaw_sensor_5, origin xyz=-0.0280979685485363 -0.027626603841781616 -0.11977264285087585 rpy=1.5915374755859375 1.0039254760840777e-08 -0.16846124827861786, axis -0.16762951016426086 -0.9856319427490234 -0.020739588886499405
- joint right_shoulder_roll_base_joint: origin xyz=-0.0342 0.2095 -0.43358 rpy=0 0 0 -> xyz=0 0 0 rpy=0 0 0
- joint right_shoulder_roll_sensor_0_joint: axis 0.977189 0.21237 0.001 -> 1.574 0.016 1.618; origin xyz=-0.033 0.049 -0.099 rpy=-1.566 -0.001 0.214 -> xyz=0.019 -0.001 0.022 rpy=-1.574 -0.072 -1.524
- joint right_shoulder_roll_sensor_1_joint: axis 0.991169 0.132608 -0.0 -> 0.095 -1.642 -2.656; origin xyz=-0.026 -0.049 -0.100 rpy=1.570 0.000 0.133 -> xyz=0.015 0.031 -0.046 rpy=-1.642 -0.107 -0.982
- joint right_shoulder_roll_sensor_2_joint: axis 0.046658 -0.996317 0.071938 -> -0.066 -1.636 2.606; origin xyz=0.017 -0.000 -0.028 rpy=-1.574 -0.072 -1.524 -> xyz=0.013 -0.034 -0.049 rpy=1.637 -0.095 0.962
- joint right_shoulder_roll_sensor_3_joint: axis 0.569302 0.816638 0.094857 -> 1.561 -0.021 1.671; origin xyz=0.012 -0.026 -0.091 rpy=1.637 -0.095 0.962 -> xyz=0.019 -0.000 -0.100 rpy=-1.561 0.100 -1.470
- joint right_shoulder_roll_sensor_4_joint: axis 0.537327 -0.836837 0.104807 -> -1.566 -0.001 0.214; origin xyz=0.008 0.032 -0.085 rpy=-1.638 -0.105 -1.000 -> xyz=-0.039 0.052 -0.112 rpy=-1.566 -0.001 0.214
- joint right_shoulder_roll_sensor_5_joint: axis 0.537327 -0.836837 0.104807 -> 1.572 0.0 -0.184; origin xyz=0.013 -0.035 -0.006 rpy=1.637 -0.095 0.964 -> xyz=-0.041 -0.052 -0.113 rpy=1.572 0.000 -0.184

File: urdf/compiled/robot_model.urdf (robot description, URDF)
Before this commit: robot h1_2, 39 links, 38 joints
Links:
- added link right_elbow_sensor_0
- added link right_elbow_sensor_1
- added link right_elbow_sensor_2
- added link right_elbow_sensor_3
- added link right_elbow_sensor_4
- added link right_elbow_sensor_5
- added link right_elbow_sensor_6
- added link right_elbow_sensor_7
- added link right_elbow_sensor_8
- added link right_elbow_skin; visual mesh filename=meshes/skin/tof/elbow_R_skin.stl scale=1 1 1
- link right_shoulder_roll_skin: geometry visual mesh filename=meshes/skin/tof/shoulder_roll_R_skin.stl scale=1 1 1
Joints:
- added joint right_elbow_base_joint: type fixed, parent right_elbow_link, child right_elbow_skin, origin xyz=0 0 0 rpy=0 0 0
- added joint right_elbow_sensor_0_joint: type fixed, parent right_elbow_skin, child right_elbow_sensor_0, origin xyz=-0.0054705264046788216 -0.01703549548983574 -0.02506975084543228 rpy=1.6108835935592651 3.0750507695742613e-10 -0.003349356586113572, axis -0.0033466597087681293 -0.9991910457611084 -0.04007663577795029
- added joint right_elbow_sensor_1_joint: type fixed, parent right_elbow_skin, child right_elbow_sensor_1, origin xyz=0.09776215255260468 -0.009773069061338902 -0.003952523693442345 rpy=1.4375799894332886 -2.939074983387968e-09 0.032789308577775955, axis 0.03249296545982361 -0.9906070828437805 0.1328226923942566
- added joint right_elbow_sensor_2_joint: type fixed, parent right_elbow_skin, child right_elbow_sensor_2, origin xyz=0.02981957234442234 -0.015662170946598053 0.0170421302318573 rpy=1.4639254808425903 -1.415918404745753e-08 0.13112856447696686, axis 0.13000711798667908 -0.9857586622238159 0.10666757822036743
- added joint right_elbow_sensor_3_joint: type fixed, parent right_elbow_skin, child right_elbow_sensor_3, origin xyz=0.03183375298976898 -0.012470245361328125 -0.038558200001716614 rpy=2.034855842590332 1.6719945428178562e-09 0.1387859433889389, axis 0.12371029704809189 -0.8856444358825684 -0.4475819766521454
- added joint right_elbow_sensor_4_joint: type fixed, parent right_elbow_skin, child right_elbow_sensor_4, origin xyz=0.09520145505666733 0.008756054565310478 0.02564341574907303 rpy=0.5687653422355652 -1.8162769066520923e-08 0.12151739746332169, axis 0.06528738886117935 -0.5346206426620483 0.8425664901733398
- added joint right_elbow_sensor_5_joint: type fixed, parent right_elbow_skin, child right_elbow_sensor_5, origin xyz=-0.006869952194392681 -0.017091382294893265 0.005429353564977646 rpy=1.5707944631576538 2.0792034760575007e-10 0.004111796617507935, axis 0.004111784510314465 -0.9999915361404419 2.02366391022224e-06
- added joint right_elbow_sensor_6_joint: type fixed, parent right_elbow_skin, child right_elbow_sensor_6, origin xyz=0.08788560330867767 0.03748124837875366 0.03188776969909668 rpy=0.10568315535783768 -2.4437664336574016e-08 3.049027919769287, axis 0.00975038856267929 0.10503476858139038 0.9944207668304443
- added joint right_elbow_sensor_7_joint: type fixed, parent right_elbow_skin, child right_elbow_sensor_7, origin xyz=0.08021856844425201 0.01752631552517414 -0.05247209593653679 rpy=2.8729567527770996 -1.6629815746682652e-08 0.188669815659523, axis 0.049779538065195084 -0.26070669293403625 -0.9641338586807251
- added joint right_elbow_sensor_8_joint: type fixed, parent right_elbow_skin, child right_elbow_sensor_8, origin xyz=0.06785736232995987 -0.006429128348827362 -0.03632089123129845 rpy=2.093989372253418 -2.5215447507775934e-09 0.17718012630939484, axis 0.15267664194107056 -0.8526670932769775 -0.4996485412120819

Commit message: added new shoulder yaw

File: urdf/compiled/h1_2_handless_tof.urdf (robot description, URDF)
Before this commit: robot h1_2, 56 links, 55 joints
Links:
- removed link left_elbow_sensor_8
- added link right_shoulder_yaw_sensor_6
Joints:
- removed joint left_elbow_sensor_8_joint
- added joint right_shoulder_yaw_sensor_6_joint: type fixed, parent right_shoulder_yaw_skin, child right_shoulder_yaw_sensor_6, origin xyz=0.049 -0.021 -0.038 rpy=1.584 -0.029 1.136, axis 1.584 -0.029 1.136
- joint left_elbow_sensor_0_joint: axis -0.0033466597087681293 -0.9991910457611084 -0.04007663577795029 -> 1.643 0.053 -0.634; origin xyz=-0.0054705264046788216 -0.01703549548983574 -0.02506975084543228 rpy=1.6108835935592651 3.0750507695742613e-10 -0.003349356586113572 -> xyz=-0.045 -0.011 -0.005 rpy=1.643 0.053 -0.634
- joint left_elbow_sensor_1_joint: axis 0.03249296545982361 -0.9906070828437805 0.1328226923942566 -> 1.078 -0.02 -0.037; origin xyz=0.09776215255260468 -0.009773069061338902 -0.003952523693442345 rpy=1.4375799894332886 -2.939074983387968e-09 0.032789308577775955 -> xyz=-0.001 -0.013 0.042 rpy=1.078 -0.020 -0.037
- joint left_elbow_sensor_2_joint: axis 0.13000711798667908 -0.9857586622238159 0.10666757822036743 -> 0.944 -3.13 0.055; origin xyz=0.02981957234442234 -0.015662170946598053 0.0170421302318573 rpy=1.4639254808425903 -1.415918404745753e-08 0.13112856447696686 -> xyz=0.002 -0.012 -0.044 rpy=2.198 -0.022 0.031
- joint left_elbow_sensor_3_joint: axis 0.12371029704809189 -0.8856444358825684 -0.4475819766521454 -> 1.572 -0.0 0.017; origin xyz=0.03183375298976898 -0.012470245361328125 -0.038558200001716614 rpy=2.034855842590332 1.6719945428178562e-09 0.1387859433889389 -> xyz=0.002 -0.017 -0.003 rpy=1.572 -0.000 0.017
- joint left_elbow_sensor_4_joint: axis 0.06528738886117935 -0.5346206426620483 0.8425664901733398 -> 1.57 0.0 0.144; origin xyz=0.09520145505666733 0.008756054565310478 0.02564341574907303 rpy=0.5687653422355652 -1.8162769066520923e-08 0.12151739746332169 -> xyz=0.048 -0.014 -0.005 rpy=1.570 0.000 0.144
- joint left_elbow_sensor_5_joint: axis 0.004111784510314465 -0.9999915361404419 2.02366391022224e-06 -> 1.542 0.0 0.017; origin xyz=-0.006869952194392681 -0.017091382294893265 0.005429353564977646 rpy=1.5707944631576538 2.0792034760575007e-10 0.004111796617507935 -> xyz=0.095 -0.010 -0.008 rpy=1.542 0.000 0.017
- joint left_elbow_sensor_6_joint: axis 0.00975038856267929 0.10503476858139038 0.9944207668304443 -> 0.179 0.036 0.007; origin xyz=0.08788560330867767 0.03748124837875366 0.03188776969909668 rpy=0.10568315535783768 -2.4437664336574016e-08 3.049027919769287 -> xyz=0.089 0.021 0.031 rpy=0.179 0.036 0.007
- joint left_elbow_sensor_7_joint: axis 0.049779538065195084 -0.26070669293403625 -0.9641338586807251 -> 3.032 -0.022 0.002; origin xyz=0.08021856844425201 0.01752631552517414 -0.05247209593653679 rpy=2.8729567527770996 -1.6629815746682652e-08 0.188669815659523 -> xyz=0.089 0.026 -0.054 rpy=3.032 -0.022 0.002
- joint right_shoulder_yaw_sensor_0_joint: axis 0.9508576989173889 -0.12113388627767563 -0.28494971990585327 -> -1.586 -0.062 1.796; origin xyz=0.04118751734495163 -0.004814512562006712 -0.08737954497337341 rpy=1.8597503900527954 1.1286831025358879e-08 1.4440847635269165 -> xyz=-0.052 -0.011 -0.040 rpy=1.586 0.067 -1.345
- joint right_shoulder_yaw_sensor_1_joint: axis -0.6932508945465088 -0.7167385220527649 -0.07542620599269867 -> 1.641 1.629 -1.218; origin xyz=-0.035796575248241425 -0.03355425223708153 -0.04064032435417175 rpy=1.646294355392456 1.8119585831755103e-09 -0.7687416672706604 -> xyz=-0.051 -0.012 -0.092 rpy=1.567 -0.014 -1.288
- joint right_shoulder_yaw_sensor_2_joint: axis 0.04019082337617874 -0.9604589939117432 -0.2755054235458374 -> -0.259 -1.757 1.398; origin xyz=0.0068807341158390045 -0.038329385221004486 -0.07258914411067963 rpy=1.8499118089675903 -2.4386073160798105e-09 0.04182104021310806 -> xyz=-0.028 -0.039 -0.069 rpy=1.751 0.082 -0.421
- joint right_shoulder_yaw_sensor_3_joint: axis -0.9944165349006653 -0.10552489757537842 -0.0004047837865073234 -> 1.39 -3.116 0.091; origin xyz=-0.04953809827566147 -0.003564621554687619 -0.0796278566122055 rpy=1.571201205253601 3.790614400145387e-08 -1.4650746583938599 -> xyz=0.006 -0.049 -0.043 rpy=1.751 -0.015 0.084
- joint right_shoulder_yaw_sensor_4_joint: axis -0.13521844148635864 0.9906842708587646 0.01614234782755375 -> 1.41 -3.101 0.006; origin xyz=-0.00878828577697277 0.04951019585132599 -0.0318453386425972 rpy=1.5546531677246094 -2.4349319005523284e-08 -3.0059409141540527 -> xyz=0.003 -0.033 -0.106 rpy=1.731 0.000 -0.001
- joint right_shoulder_yaw_sensor_5_joint: axis -0.16762951016426086 -0.9856319427490234 -0.020739588886499405 -> 1.814 0.018 0.641; origin xyz=-0.0280979685485363 -0.027626603841781616 -0.11977264285087585 rpy=1.5915374755859375 1.0039254760840777e-08 -0.16846124827861786 -> xyz=0.032 -0.034 -0.072 rpy=1.818 -0.171 0.594

Commit message: add meshes

File: urdf/compiled/h1_2_handless_tof.urdf (robot description, URDF)
Before this commit: robot h1_2, 56 links, 55 joints
Links:
- added link left_shoulder_roll_sensor_0
- added link left_shoulder_roll_sensor_1
- added link left_shoulder_roll_sensor_2
- added link left_shoulder_roll_sensor_3
- added link left_shoulder_roll_sensor_4
- added link left_shoulder_roll_sensor_5
- added link left_shoulder_roll_skin; visual mesh filename=package://gentact_ros_tools_hybrid/meshes/h1_2/skin/tof/sho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 scale=1 1 1
Joints:
- added joint left_shoulder_roll_base_joint: type fixed, parent left_shoulder_roll_link, child left_shoulder_roll_skin, origin xyz=0 0 0 rpy=0 0 0
- added joint left_shoulder_roll_sensor_0_joint: type fixed, parent left_shoulder_roll_skin, child left_shoulder_roll_sensor_0, origin xyz=0.019 -0.001 0.022 rpy=-1.574 -0.072 -1.524, axis 1.574 0.016 1.618
- added joint left_shoulder_roll_sensor_1_joint: type fixed, parent left_shoulder_roll_skin, child left_shoulder_roll_sensor_1, origin xyz=0.015 0.031 -0.046 rpy=-1.642 -0.107 -0.982, axis 0.095 -1.642 -2.656
- added joint left_shoulder_roll_sensor_2_joint: type fixed, parent left_shoulder_roll_skin, child left_shoulder_roll_sensor_2, origin xyz=0.013 -0.034 -0.049 rpy=1.637 -0.095 0.962, axis -0.066 -1.636 2.606
- added joint left_shoulder_roll_sensor_3_joint: type fixed, parent left_shoulder_roll_skin, child left_shoulder_roll_sensor_3, origin xyz=0.019 -0.000 -0.100 rpy=-1.561 0.100 -1.470, axis 1.561 -0.021 1.671
- added joint left_shoulder_roll_sensor_4_joint: type fixed, parent left_shoulder_roll_skin, child left_shoulder_roll_sensor_4, origin xyz=-0.039 0.052 -0.112 rpy=-1.566 -0.001 0.214, axis -1.566 -0.001 0.214
- added joint left_shoulder_roll_sensor_5_joint: type fixed, parent left_shoulder_roll_skin, child left_shoulder_roll_sensor_5, origin xyz=-0.041 -0.052 -0.113 rpy=1.572 0.000 -0.184, axis 1.572 0.0 -0.184
