Commit message: add more h1-2 skins

File: urdf/compiled/h1_2_handless_tof.urdf (robot description, URDF)
Before this commit: robot h1_2, 63 links, 62 joints
Links:
- removed link right_shoulder_yaw_sensor_6
- added link head_sensor_0
- added link head_sensor_1
- added link head_sensor_2
- added link head_sensor_3
- added link head_sensor_4
- added link head_skin; visual mesh filename=package://gentact_ros_tools_hybrid/meshes/h1_2/skin/tof/hea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 scale=1 1 1
- added link left_hip_roll_sensor_0
- added link left_hip_roll_sensor_1
- added link left_hip_roll_sensor_2
- added link left_hip_roll_sensor_3
- added link left_hip_roll_sensor_4
- added link left_hip_roll_sensor_5
- added link left_hip_roll_sensor_6
- added link left_hip_roll_sensor_7
- added link left_hip_roll_skin; visual mesh filename=package://gentact_ros_tools_hybrid/meshes/h1_2/skin/tof/lef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 scale=1 1 1
- added link left_knee_sensor_0
- added link left_knee_sensor_1
- added link left_knee_sensor_2
- added link left_knee_sensor_3
- added link left_knee_sensor_4
- added link left_knee_skin; visual mesh filename=package://gentact_ros_tools_hybrid/meshes/h1_2/skin/tof/lef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 scale=1 1 1
- added link left_shoulder_yaw_sensor_0
- added link left_shoulder_yaw_sensor_1
- added link left_shoulder_yaw_sensor_2
- added link left_shoulder_yaw_sensor_3
- added link left_shoulder_yaw_sensor_4
- added link left_shoulder_yaw_sensor_5
- added link left_shoulder_yaw_skin; visual mesh filename=package://gentact_ros_tools_hybrid/meshes/h1_2/skin/tof/lef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 scale=1 1 1
- added link right_elbow_sensor_0
- added link right_elbow_sensor_1
- added link right_elbow_sensor_2
- added link right_elbow_sensor_3
- added link right_elbow_sensor_4
- added link right_elbow_sensor_5
- added link right_elbow_sensor_6
- added link right_elbow_sensor_7
- added link right_elbow_skin; visual mesh filename=package://gentact_ros_tools_hybrid/meshes/h1_2/skin/tof/rig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 scale=1 1 1
- added link right_hip_roll_sensor_0
- added link right_hip_roll_sensor_1
- added link right_hip_roll_sensor_2
- added link right_hip_roll_sensor_3
- added link right_hip_roll_sensor_4
- added link right_hip_roll_sensor_5
- added link right_hip_roll_sensor_6
- added link right_hip_roll_sensor_7
- added link right_hip_roll_skin; visual mesh filename=package://gentact_ros_tools_hybrid/meshes/h1_2/skin/tof/rig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 scale=1 1 1
- added link right_knee_sensor_0
- added link right_knee_sensor_1
- added link right_knee_sensor_2
- added link right_knee_sensor_3
- added link right_knee_sensor_4
- added link right_knee_skin; visual mesh filename=package://gentact_ros_tools_hybrid/meshes/h1_2/skin/tof/rig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 scale=1 1 1
- link left_ankle_pitch_link: geometry visual mesh filename=package://gentact_ros_tools_hybrid/meshes/h1_2//left_ankle_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
- link left_ankle_roll_link: geometry collision mesh filename=package://gentact_ros_tools_hybrid/meshes/h1_2//left_ankle_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; visual mesh filename=package://gentact_ros_tools_hybrid/meshes/h1_2//left_ankle_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
- link left_elbow_link: geometry collision mesh filename=package://gentact_ros_tools_hybrid/meshes/h1_2//left_elbow_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; visual mesh filename=package://gentact_ros_tools_hybrid/meshes/h1_2//left_elbow_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
- link left_hip_pitch_link: geometry collision mesh filename=package://gentact_ros_tools_hybrid/meshes/h1_2//left_hip_pi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; visual mesh filename=package://gentact_ros_tools_hybrid/meshes/h1_2//left_hip_pi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
- link left_hip_roll_link: geometry collision mesh filename=package://gentact_ros_tools_hybrid/meshes/h1_2//left_hip_ro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; visual mesh filename=package://gentact_ros_tools_hybrid/meshes/h1_2//left_hip_ro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
- link left_hip_yaw_link: geometry visual mesh filename=package://gentact_ros_tools_hybrid/meshes/h1_2//left_hip_ya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
- link left_knee_link: geometry collision cylinder length=0.2 radius=0.04; visual mesh filename=package://gentact_ros_tools_hybrid/meshes/h1_2//left_knee_l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
- link left_shoulder_pitch_link: geometry collision mesh filename=package://gentact_ros_tools_hybrid/meshes/h1_2//left_should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; visual mesh filename=package://gentact_ros_tools_hybrid/meshes/h1_2//left_should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
- link left_shoulder_roll_link: geometry collision mesh filename=package://gentact_ros_tools_hybrid/meshes/h1_2//left_should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; visual mesh filename=package://gentact_ros_tools_hybrid/meshes/h1_2//left_should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
- link left_shoulder_yaw_link: geometry collision mesh filename=package://gentact_ros_tools_hybrid/meshes/h1_2//left_should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; visual mesh filename=package://gentact_ros_tools_hybrid/meshes/h1_2//left_should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
- link left_wrist_pitch_link: geometry collision mesh filename=package://gentact_ros_tools_hybrid/meshes/h1_2//left_wrist_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; visual mesh filename=package://gentact_ros_tools_hybrid/meshes/h1_2//left_wrist_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
- link left_wrist_roll_link: geometry collision mesh filename=package://gentact_ros_tools_hybrid/meshes/h1_2//left_wrist_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; visual mesh filename=package://gentact_ros_tools_hybrid/meshes/h1_2//left_wrist_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
- link left_wrist_yaw_link: geometry visual mesh filename=package://gentact_ros_tools_hybrid/meshes/h1_2//wrist_yaw_l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
- link logo_link: geometry visual mesh filename=package://gentact_ros_tools_hybrid/meshes/h1_2//logo_link.S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
- link pelvis: geometry collision mesh filename=package://gentact_ros_tools_hybrid/meshes/h1_2//pelvis.STL; visual mesh filename=package://gentact_ros_tools_hybrid/meshes/h1_2//pelvis.STL
- link right_ankle_pitch_link: geometry visual mesh filename=package://gentact_ros_tools_hybrid/meshes/h1_2//right_ankle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
- link right_ankle_roll_link: geometry collision mesh filename=package://gentact_ros_tools_hybrid/meshes/h1_2//right_ankle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; visual mesh filename=package://gentact_ros_tools_hybrid/meshes/h1_2//right_ankle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
- link right_elbow_link: geometry collision mesh filename=package://gentact_ros_tools_hybrid/meshes/h1_2//right_elbow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; visual mesh filename=package://gentact_ros_tools_hybrid/meshes/h1_2//right_elbow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
- link right_hip_pitch_link: geometry collision mesh filename=package://gentact_ros_tools_hybrid/meshes/h1_2//right_hip_p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; visual mesh filename=package://gentact_ros_tools_hybrid/meshes/h1_2//right_hip_p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
- link right_hip_roll_link: geometry collision mesh filename=package://gentact_ros_tools_hybrid/meshes/h1_2//right_hip_r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; visual mesh filename=package://gentact_ros_tools_hybrid/meshes/h1_2//right_hip_r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
- link right_hip_yaw_link: geometry visual mesh filename=package://gentact_ros_tools_hybrid/meshes/h1_2//right_hip_y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
- link right_knee_link: geometry collision cylinder length=0.2 radius=0.04; visual mesh filename=package://gentact_ros_tools_hybrid/meshes/h1_2//right_knee_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
- link right_shoulder_pitch_link: geometry collision mesh filename=package://gentact_ros_tools_hybrid/meshes/h1_2//right_shoul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; visual mesh filename=package://gentact_ros_tools_hybrid/meshes/h1_2//right_shoul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
- link right_shoulder_roll_link: geometry collision mesh filename=package://gentact_ros_tools_hybrid/meshes/h1_2//right_shoul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; visual mesh filename=package://gentact_ros_tools_hybrid/meshes/h1_2//right_shoul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
- link right_shoulder_yaw_link: geometry collision mesh filename=package://gentact_ros_tools_hybrid/meshes/h1_2//right_shoul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; visual mesh filename=package://gentact_ros_tools_hybrid/meshes/h1_2//right_shoul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
- link right_wrist_pitch_link: geometry collision mesh filename=package://gentact_ros_tools_hybrid/meshes/h1_2//right_wrist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; visual mesh filename=package://gentact_ros_tools_hybrid/meshes/h1_2//right_wrist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
- link right_wrist_roll_link: geometry collision mesh filename=package://gentact_ros_tools_hybrid/meshes/h1_2//right_wrist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; visual mesh filename=package://gentact_ros_tools_hybrid/meshes/h1_2//right_wrist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
- link right_wrist_yaw_link: geometry visual mesh filename=package://gentact_ros_tools_hybrid/meshes/h1_2//wrist_yaw_l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
- link torso_link: geometry collision mesh filename=package://gentact_ros_tools_hybrid/meshes/h1_2//torso_link.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; visual mesh filename=package://gentact_ros_tools_hybrid/meshes/h1_2//torso_link.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
Joints:
- removed joint right_shoulder_yaw_sensor_6_joint
- added joint head_base_joint: type fixed, parent torso_link, child head_skin, origin xyz=0 0 0 rpy=0 0 0
- added joint head_sensor_0_joint: type fixed, parent head_skin, child head_sensor_0, origin xyz=0.049 0.001 0.775 rpy=0.005 0.033 0.000, axis 0.032994 -0.005 0.999443
- added joint head_sensor_1_joint: type fixed, parent head_skin, child head_sensor_1, origin xyz=0.129 0.003 0.721 rpy=-0.013 1.155 -0.012, axis 0.914808 0.002022 0.403884
- added joint head_sensor_2_joint: type fixed, parent head_skin, child head_sensor_2, origin xyz=0.059 -0.069 0.741 rpy=1.048 0.109 0.187, axis 0.214449 -0.841223 0.496342
- added joint head_sensor_3_joint: type fixed, parent head_skin, child head_sensor_3, origin xyz=-0.029 -0.003 0.744 rpy=0.386 -0.878 -0.303, axis -0.792712 -0.146632 0.591698
- added joint head_sensor_4_joint: type fixed, parent head_skin, child head_sensor_4, origin xyz=0.044 0.070 0.743 rpy=-1.018 -0.011 0.017, axis -0.020242 0.850838 0.525037
- added joint left_hip_roll_base_joint: type fixed, parent left_hip_roll_link, child left_hip_roll_skin, origin xyz=0 0 0 rpy=0 0 0
- added joint left_hip_roll_sensor_0_joint: type fixed, parent left_hip_roll_skin, child left_hip_roll_sensor_0, origin xyz=0.006 0.079 -0.118 rpy=-1.610 -0.003 -0.072, axis 0.072 0.996634 -0.039193
- added joint left_hip_roll_sensor_1_joint: type fixed, parent left_hip_roll_skin, child left_hip_roll_sensor_1, origin xyz=0.036 0.078 -0.041 rpy=-1.597 -0.004 -0.141, axis 0.140589 0.989721 -0.0262
- added joint left_hip_roll_sensor_2_joint: type fixed, parent left_hip_roll_skin, child left_hip_roll_sensor_2, origin xyz=-0.007 0.083 -0.000 rpy=-1.597 0.001 0.046, axis -0.045994 0.998598 -0.026201
- added joint left_hip_roll_sensor_3_joint: type fixed, parent left_hip_roll_skin, child left_hip_roll_sensor_3, origin xyz=0.068 0.017 -0.061 rpy=-1.699 -1.122 -1.428, axis 0.998092 0.027125 -0.055473
- added joint left_hip_roll_sensor_4_joint: type fixed, parent left_hip_roll_skin, child left_hip_roll_sensor_4, origin xyz=0.071 0.043 0.003 rpy=-1.659 -0.882 -1.457, axis 0.997392 0.045543 -0.05599
- added joint left_hip_roll_sensor_5_joint: type fixed, parent left_hip_roll_skin, child left_hip_roll_sensor_5, origin xyz=0.064 0.043 -0.122 rpy=-1.699 -1.122 -1.428, axis 0.998092 0.027125 -0.055473
- added joint left_hip_roll_sensor_6_joint: type fixed, parent left_hip_roll_skin, child left_hip_roll_sensor_6, origin xyz=-0.080 0.025 -0.009 rpy=-2.077 1.370 1.056, axis -0.995167 0.017072 -0.096705
- added joint left_hip_roll_sensor_7_joint: type fixed, parent left_hip_roll_skin, child left_hip_roll_sensor_7, origin xyz=-0.063 0.027 -0.089 rpy=-2.571 1.371 0.562, axis -0.985797 0.017514 -0.167028
- added joint left_knee_base_joint: type fixed, parent left_knee_link, child left_knee_skin, origin xyz=0 0 0 rpy=0 0 0
- added joint left_knee_sensor_0_joint: type fixed, parent left_knee_skin, child left_knee_sensor_0, origin xyz=0.061 -0.034 0.026 rpy=3.142 -1.556 0.000, axis 0.015314 0.000908 0.999882
- added joint left_knee_sensor_1_joint: type fixed, parent left_knee_skin, child left_knee_sensor_1, origin xyz=0.060 0.003 -0.025 rpy=3.142 -1.537 0.000, axis -0.034685 -0.00091 -0.999398
- added joint left_knee_sensor_2_joint: type fixed, parent left_knee_skin, child left_knee_sensor_2, origin xyz=0.058 0.005 -0.073 rpy=3.142 -1.537 0.000, axis 0.996841 0.003415 -0.079347
- added joint left_knee_sensor_3_joint: type fixed, parent left_knee_skin, child left_knee_sensor_3, origin xyz=0.013 0.055 0.012 rpy=-1.571 0.000 0.000, axis -3.3e-05 1.0 -0.000906
- added joint left_knee_sensor_4_joint: type fixed, parent left_knee_skin, child left_knee_sensor_4, origin xyz=0.010 0.055 -0.063 rpy=-1.544 -0.000 0.007, axis -0.005593 0.994921 -0.100504
- added joint left_shoulder_yaw_base_joint: type fixed, parent left_shoulder_yaw_link, child left_shoulder_yaw_skin, origin xyz=0 0 0 rpy=0 0 0
- added joint left_shoulder_yaw_sensor_0_joint: type fixed, parent left_shoulder_yaw_skin, child left_shoulder_yaw_sensor_0, origin xyz=0.031 0.034 -0.032 rpy=-1.633 -0.056 -0.731, axis 0.668914 0.740744 -0.062066
- added joint left_shoulder_yaw_sensor_1_joint: type fixed, parent left_shoulder_yaw_skin, child left_shoulder_yaw_sensor_1, origin xyz=-0.006 0.044 -0.034 rpy=-1.713 0.008 0.057, axis -0.057526 0.988234 -0.14172
- added joint left_shoulder_yaw_sensor_2_joint: type fixed, parent left_shoulder_yaw_skin, child left_shoulder_yaw_sensor_2, origin xyz=-0.016 0.034 -0.073 rpy=-1.832 0.024 0.089, axis -0.09204 0.961705 -0.258169
- added joint left_shoulder_yaw_sensor_3_joint: type fixed, parent left_shoulder_yaw_skin, child left_shoulder_yaw_sensor_3, origin xyz=-0.045 0.011 -0.035 rpy=-1.572 0.003 1.343, axis -0.974167 0.225828 -0.001204
- added joint left_shoulder_yaw_sensor_4_joint: type fixed, parent left_shoulder_yaw_skin, child left_shoulder_yaw_sensor_4, origin xyz=-0.046 -0.002 -0.097 rpy=3.142 1.571 0.000, axis -1.0 0.000407 0.000204
- added joint left_shoulder_yaw_sensor_5_joint: type fixed, parent left_shoulder_yaw_skin, child left_shoulder_yaw_sensor_5, origin xyz=-0.021 -0.042 -0.029 rpy=1.536 -0.016 -0.427, axis -0.414398 -0.909431 0.034785
- added joint right_elbow_base_joint: type fixed, parent right_elbow_link, child right_elbow_skin, origin xyz=0 0 0 rpy=0 0 0
- added joint right_elbow_sensor_0_joint: type fixed, parent right_elbow_skin, child right_elbow_sensor_0, origin xyz=-0.045 -0.011 -0.005 rpy=1.643 0.053 -0.634, axis -0.593908 -0.801301 -0.07204
- added joint right_elbow_sensor_1_joint: type fixed, parent right_elbow_skin, child right_elbow_sensor_1, origin xyz=-0.001 -0.013 0.042 rpy=1.078 -0.020 -0.037, axis -0.042045 -0.88006 0.472997
- added joint right_elbow_sensor_2_joint: type fixed, parent right_elbow_skin, child right_elbow_sensor_2, origin xyz=0.002 -0.012 -0.044 rpy=2.198 -0.022 0.031, axis 0.038 -0.808883 -0.586741
- added joint right_elbow_sensor_3_joint: type fixed, parent right_elbow_skin, child right_elbow_sensor_3, origin xyz=0.002 -0.017 -0.003 rpy=1.572 0.000 0.017, axis 0.016999 -0.999855 -0.001204
- added joint right_elbow_sensor_4_joint: type fixed, parent right_elbow_skin, child right_elbow_sensor_4, origin xyz=0.048 -0.014 -0.005 rpy=1.570 0.000 0.144, axis 0.143503 -0.98965 0.000796
- added joint right_elbow_sensor_5_joint: type fixed, parent right_elbow_skin, child right_elbow_sensor_5, origin xyz=0.095 -0.010 -0.008 rpy=1.542 0.000 0.017, axis 0.016992 -0.999441 0.028792
- added joint right_elbow_sensor_6_joint: type fixed, parent right_elbow_skin, child right_elbow_sensor_6, origin xyz=0.089 0.021 0.031 rpy=0.179 0.036 0.007, axis 0.036663 -0.177793 0.983385
- added joint right_elbow_sensor_7_joint: type fixed, parent right_elbow_skin, child right_elbow_sensor_7, origin xyz=0.089 0.026 -0.054 rpy=3.032 -0.022 0.002, axis 0.022085 -0.109329 -0.99376
- added joint right_hip_roll_base_joint: type fixed, parent right_hip_roll_link, child right_hip_roll_skin, origin xyz=0 0 0 rpy=0 0 0
- added joint right_hip_roll_sensor_0_joint: type fixed, parent right_hip_roll_skin, child right_hip_roll_sensor_0, origin xyz=0.006 -0.079 -0.118 rpy=1.610 -0.003 0.072, axis -0.042383 -0.997948 -0.047987
- added joint right_hip_roll_sensor_1_joint: type fixed, parent right_hip_roll_skin, child right_hip_roll_sensor_1, origin xyz=0.036 -0.078 -0.041 rpy=1.597 -0.004 0.141, axis 0.141961 -0.989671 -0.01994
- added joint right_hip_roll_sensor_2_joint: type fixed, parent right_hip_roll_skin, child right_hip_roll_sensor_2, origin xyz=-0.007 -0.083 0.000 rpy=1.597 0.001 -0.046, axis -0.998868 0.044535 -0.016738
- added joint right_hip_roll_sensor_3_joint: type fixed, parent right_hip_roll_skin, child right_hip_roll_sensor_3, origin xyz=0.068 -0.017 -0.061 rpy=1.699 -1.122 1.428, axis 0.999652 -0.026273 -0.002366
- added joint right_hip_roll_sensor_4_joint: type fixed, parent right_hip_roll_skin, child right_hip_roll_sensor_4, origin xyz=0.071 -0.043 0.003 rpy=1.659 -0.882 1.457, axis 0.998938 -0.045993 -0.002585
- added joint right_hip_roll_sensor_5_joint: type fixed, parent right_hip_roll_skin, child right_hip_roll_sensor_5, origin xyz=0.064 -0.043 -0.122 rpy=1.699 -1.122 1.428, axis 0.999652 -0.026273 -0.002366
- added joint right_hip_roll_sensor_6_joint: type fixed, parent right_hip_roll_skin, child right_hip_roll_sensor_6, origin xyz=-0.080 -0.025 -0.009 rpy=2.077 1.370 -1.056, axis -0.995585 -0.018047 -0.092116
- added joint right_hip_roll_sensor_7_joint: type fixed, parent right_hip_roll_skin, child right_hip_roll_sensor_7, origin xyz=-0.063 -0.027 -0.089 rpy=2.571 1.371 -0.562, axis -0.951851 -0.016972 -0.30609
- added joint right_knee_base_joint: type fixed, parent right_knee_link, child right_knee_skin, origin xyz=0 0 0 rpy=0 0 0
- added joint right_knee_sensor_0_joint: type fixed, parent right_knee_skin, child right_knee_sensor_0, origin xyz=0.057 0.034 -0.132 rpy=1.7383 0.0000 1.6544, axis 0.982561 0.082325 -0.166725
- added joint right_knee_sensor_1_joint: type fixed, parent right_knee_skin, child right_knee_sensor_1, origin xyz=0.057 -0.003 -0.184 rpy=1.6613 0.0000 1.5710, axis 0.995909 0.000227 -0.090357
- added joint right_knee_sensor_2_joint: type fixed, parent right_knee_skin, child right_knee_sensor_2, origin xyz=0.056 -0.005 -0.231 rpy=1.6613 0.0000 1.5710, axis 0.995909 0.000227 -0.090357
- added joint right_knee_sensor_3_joint: type fixed, parent right_knee_skin, child right_knee_sensor_3, origin xyz=0.010 -0.055 -0.146 rpy=1.5699 0.0000 0.0000, axis 3.3e-05 -1.0 0.000906
- added joint right_knee_sensor_4_joint: type fixed, parent right_knee_skin, child right_knee_sensor_4, origin xyz=0.007 -0.055 -0.221 rpy=1.6697 0.0000 -0.0056, axis -0.005527 -0.995102 -0.098699
- joint left_elbow_sensor_0_joint: axis 1.643 0.053 -0.634 -> -0.593908 0.801301 -0.07204; origin xyz=-0.045 -0.011 -0.005 rpy=1.643 0.053 -0.634 -> xyz=-0.045 0.011 -0.005 rpy=-1.643 0.053 0.634
- joint left_elbow_sensor_1_joint: axis 1.078 -0.02 -0.037 -> -0.042045 0.88006 0.472997; origin xyz=-0.001 -0.013 0.042 rpy=1.078 -0.020 -0.037 -> xyz=-0.001 0.013 0.042 rpy=-1.078 -0.020 0.037
- joint left_elbow_sensor_2_joint: axis 0.944 -3.13 0.055 -> 0.038 0.808883 -0.586741; origin xyz=0.002 -0.012 -0.044 rpy=2.198 -0.022 0.031 -> xyz=0.002 0.012 -0.044 rpy=-2.198 -0.022 -0.031
- joint left_elbow_sensor_3_joint: axis 1.572 -0.0 0.017 -> 0.016999 0.999855 -0.001204; origin xyz=0.002 -0.017 -0.003 rpy=1.572 -0.000 0.017 -> xyz=0.002 0.017 -0.003 rpy=-1.572 0.000 -0.017
- joint left_elbow_sensor_4_joint: axis 1.57 0.0 0.144 -> 0.143503 0.98965 0.000796; origin xyz=0.048 -0.014 -0.005 rpy=1.570 0.000 0.144 -> xyz=0.048 0.014 -0.005 rpy=-1.570 0.000 -0.144
- joint left_elbow_sensor_5_joint: axis 1.542 0.0 0.017 -> 0.016992 0.999441 0.028792; origin xyz=0.095 -0.010 -0.008 rpy=1.542 0.000 0.017 -> xyz=0.095 0.010 -0.008 rpy=-1.542 0.000 -0.017
- joint left_elbow_sensor_6_joint: axis 0.179 0.036 0.007 -> 0.036663 0.177793 0.983385; origin xyz=0.089 0.021 0.031 rpy=0.179 0.036 0.007 -> xyz=0.089 -0.021 0.031 rpy=-0.179 0.036 -0.007
- joint left_elbow_sensor_7_joint: axis 3.032 -0.022 0.002 -> 0.022085 0.109329 -0.99376; origin xyz=0.089 0.026 -0.054 rpy=3.032 -0.022 0.002 -> xyz=0.089 -0.026 -0.054 rpy=-3.032 -0.022 -0.002
- joint left_shoulder_roll_sensor_0_joint: axis 1.574 0.016 1.618 -> 0.046658 -0.996317 0.071938
- joint left_shoulder_roll_sensor_1_joint: axis 0.095 -1.642 -2.656 -> 0.552184 -0.826854 0.106796
- joint left_shoulder_roll_sensor_2_joint: axis -0.066 -1.636 2.606 -> 0.569302 0.816638 0.094857
- joint left_shoulder_roll_sensor_3_joint: axis 1.561 -0.021 1.671 -> 0.100123 -0.989954 -0.099833; origin xyz=0.019 -0.000 -0.100 rpy=-1.561 0.100 -1.470 -> xyz=0.019 0.000 -0.100 rpy=-1.561 0.100 -1.470
- joint left_shoulder_roll_sensor_4_joint: axis -1.566 -0.001 0.214 -> 0.977189 0.21237 0.001
- joint left_shoulder_roll_sensor_5_joint: axis 1.572 0.0 -0.184 -> 0.98312 -0.182964 0.0
- joint right_shoulder_roll_sensor_0_joint: axis 1.574 0.016 1.618 -> 0.046658 -0.996317 0.071938
- joint right_shoulder_roll_sensor_1_joint: axis 0.095 -1.642 -2.656 -> 0.552184 -0.826854 0.106796
- joint right_shoulder_roll_sensor_2_joint: axis -0.066 -1.636 2.606 -> 0.569302 0.816638 0.094857
- joint right_shoulder_roll_sensor_3_joint: axis 1.561 -0.021 1.671 -> 0.100123 -0.989954 -0.099833; origin xyz=0.019 -0.000 -0.100 rpy=-1.561 0.100 -1.470 -> xyz=0.019 0.000 -0.100 rpy=-1.561 0.100 -1.470
- joint right_shoulder_roll_sensor_4_joint: axis -1.566 -0.001 0.214 -> 0.977189 0.21237 0.001
- joint right_shoulder_roll_sensor_5_joint: axis 1.572 0.0 -0.184 -> 0.98312 -0.182964 0.0
- joint right_shoulder_yaw_sensor_0_joint: axis -1.586 -0.062 1.796 -> 0.668914 -0.740744 -0.062066; origin xyz=-0.052 -0.011 -0.040 rpy=1.586 0.067 -1.345 -> xyz=0.031 -0.034 -0.032 rpy=1.633 -0.056 0.731
- joint right_shoulder_yaw_sensor_1_joint: axis 1.641 1.629 -1.218 -> -0.057526 -0.988234 -0.14172; origin xyz=-0.051 -0.012 -0.092 rpy=1.567 -0.014 -1.288 -> xyz=-0.006 -0.044 -0.034 rpy=1.713 0.008 -0.057
- joint right_shoulder_yaw_sensor_2_joint: axis -0.259 -1.757 1.398 -> -0.09204 -0.961705 -0.258169; origin xyz=-0.028 -0.039 -0.069 rpy=1.751 0.082 -0.421 -> xyz=-0.016 -0.034 -0.073 rpy=1.832 0.024 -0.089
- joint right_shoulder_yaw_sensor_3_joint: axis 1.39 -3.116 0.091 -> -0.974167 -0.225828 -0.001204; origin xyz=0.006 -0.049 -0.043 rpy=1.751 -0.015 0.084 -> xyz=-0.045 -0.011 -0.035 rpy=1.572 0.003 -1.343
- joint right_shoulder_yaw_sensor_4_joint: axis 1.41 -3.101 0.006 -> -1.0 -0.000407 0.000204; origin xyz=0.003 -0.033 -0.106 rpy=1.731 0.000 -0.001 -> xyz=-0.046 0.002 -0.097 rpy=-3.142 1.571 0.000
- joint right_shoulder_yaw_sensor_5_joint: axis 1.814 0.018 0.641 -> -0.414398 0.909431 0.034785; origin xyz=0.032 -0.034 -0.072 rpy=1.818 -0.171 0.594 -> xyz=-0.021 0.042 -0.029 rpy=-1.536 -0.016 0.427
