Commit message: new xacro

File: urdf/skin/link5.xacro (robot description, xacro)
@@ -5,5 +5,5 @@
     <!-- Properties -->
     <xacro:property name="use_mesh_file" value="true" />
-    <xacro:property name="mesh_file" value="package://gentact_ros_tools/meshes/skin/link5.stl" />
+    <xacro:property name="mesh_file" value="package://gentact_ros_tools/meshes/skin/self-cap/link5_fancy.stl" />
     <xacro:property name="mass" value="0.3" /> <!-- [kg] -->
     <xacro:property name="body_width" value="0.3" /> <!-- [m] -->
