Commit message: Working launch

File: urdf/skin/link5_fancy.xacro (robot description, xacro)
@@ -10,5 +10,5 @@
     <xacro:property name="body_height" value="0.1" /> <!-- [m] -->
     <xacro:property name="sensor_length" value="0.05" /> <!-- [m] -->
-    <xacro:property name="sensor_radius" value="0.005" /> <!-- [m] -->
+    <xacro:property name="sensor_radius" value="0.0" /> <!-- [m] -->
     <!-- Included URDF Files -->
     <xacro:include filename="$(find gentact_ros_tools)/urdf/skin/self-cap-base.xacro" />

File: urdf/skin/link6_fancy.xacro (robot description, xacro)
@@ -10,5 +10,5 @@
     <xacro:property name="body_height" value="0.1" /> <!-- [m] -->
     <xacro:property name="sensor_length" value="0.05" /> <!-- [m] -->
-    <xacro:property name="sensor_radius" value="0.005" /> <!-- [m] -->
+    <xacro:property name="sensor_radius" value="0.0" /> <!-- [m] -->
     <!-- Included URDF Files -->
     <xacro:include filename="$(find gentact_ros_tools)/urdf/skin/self-cap-base.xacro" />
@@ -29,5 +29,5 @@
       parent="${namespace}_skin"
       sensor_number="0"
-      sensor_radius="0.0"
+      sensor_radius="${sensor_radius}"
       sensor_length="0.057"
       normal_x="0.474"
@@ -40,5 +40,5 @@
       parent="${namespace}_skin"
       sensor_number="1"
-      sensor_radius="0.0"
+      sensor_radius="${sensor_radius}"
       sensor_length="0.048"
       normal_x="0.885"
@@ -51,5 +51,5 @@
       parent="${namespace}_skin"
       sensor_number="2"
-      sensor_radius="0.0"
+      sensor_radius="${sensor_radius}"
       sensor_length="0.060"
       normal_x="0.991"
@@ -62,5 +62,5 @@
       parent="${namespace}_skin"
       sensor_number="3"
-      sensor_radius="0.0"
+      sensor_radius="${sensor_radius}"
       sensor_length="0.059"
       normal_x="0.477"
@@ -73,5 +73,5 @@
       parent="${namespace}_skin"
       sensor_number="4"
-      sensor_radius="0.0"
+      sensor_radius="${sensor_radius}"
       sensor_length="0.059"
       normal_x="0.888"
@@ -84,5 +84,5 @@
       parent="${namespace}_skin"
       sensor_number="5"
-      sensor_radius="0.0"
+      sensor_radius="${sensor_radius}"
       sensor_length="0.025"
       normal_x="0.995"
@@ -95,5 +95,5 @@
       parent="${namespace}_skin"
       sensor_number="6"
-      sensor_radius="0.0"
+      sensor_radius="${sensor_radius}"
       sensor_length="0.023"
       normal_x="0.776"
@@ -106,5 +106,5 @@
       parent="${namespace}_skin"
       sensor_number="7"
-      sensor_radius="0.0"
+      sensor_radius="${sensor_radius}"
       sensor_length="0.023"
       normal_x="-0.092"
