Commit message: Added link 1

File: urdf/skin/link2_fancy.xacro (robot description, xacro)
@@ -22,5 +22,5 @@
       use_mesh_file="${use_mesh_file}"
       mesh_file="${mesh_file}">
-      <origin xyz="0 0 0" rpy="0 0 0" />
+      <origin xyz="0 0 0" rpy="1.5707 0 0" />
     </xacro:dermis_base_macro>
     <!-- Instantiate sensors -->
