Commit message: Uh oh, big push here

File: urdf/skin/link3_fancy.xacro (robot description, xacro)
@@ -28,5 +28,5 @@
       robot_namespace="${namespace}"
       parent="${namespace}_skin"
-      sensor_number="5"
+      sensor_number="0"
       sensor_radius="${sensor_radius}"
       sensor_length="0.05"
@@ -39,5 +39,5 @@
       robot_namespace="${namespace}"
       parent="${namespace}_skin"
-      sensor_number="6"
+      sensor_number="1"
       sensor_radius="${sensor_radius}"
       sensor_length="0.05"
@@ -50,5 +50,5 @@
       robot_namespace="${namespace}"
       parent="${namespace}_skin"
-      sensor_number="0"
+      sensor_number="2"
       sensor_radius="${sensor_radius}"
       sensor_length="0.05"
@@ -61,5 +61,5 @@
       robot_namespace="${namespace}"
       parent="${namespace}_skin"
-      sensor_number="7"
+      sensor_number="3"
       sensor_radius="${sensor_radius}"
       sensor_length="0.05"
@@ -83,5 +83,5 @@
       robot_namespace="${namespace}"
       parent="${namespace}_skin"
-      sensor_number="3"
+      sensor_number="5"
       sensor_radius="${sensor_radius}"
       sensor_length="0.05"
@@ -94,5 +94,5 @@
       robot_namespace="${namespace}"
       parent="${namespace}_skin"
-      sensor_number="1"
+      sensor_number="6"
       sensor_radius="${sensor_radius}"
       sensor_length="0.05"
@@ -105,5 +105,5 @@
       robot_namespace="${namespace}"
       parent="${namespace}_skin"
-      sensor_number="2"
+      sensor_number="7"
       sensor_radius="${sensor_radius}"
       sensor_length="0.05"

File: urdf/skin/link6_fancy.xacro (robot description, xacro)
@@ -5,5 +5,5 @@
     <!-- Properties -->
     <xacro:property name="use_mesh_file" value="true" />
-    <xacro:property name="mesh_file" value="package://gentact_ros_tools/meshes/skin/self-cap/link6_fancy.stl" />
+    <xacro:property name="mesh_file" value="package://gentact_ros_tools/meshes/skin/link6_fancy.stl" />
     <xacro:property name="mass" value="0.3" /> <!-- [kg] -->
     <xacro:property name="body_width" value="0.3" /> <!-- [m] -->
