Commit message: created avoidance config, changed cam serial nums

File: urdf/skin/link6_fancy.xacro (robot description, xacro)
@@ -5,5 +5,5 @@
     <!-- Properties -->
     <xacro:property name="use_mesh_file" value="true" />
-    <xacro:property name="mesh_file" value="package://gentact_ros_tools/meshes/skin/link6_fancy.stl" />
+    <xacro:property name="mesh_file" value="package://gentact_ros_tools/meshes/skin/self-cap/link6_fancy.stl" />
     <xacro:property name="mass" value="0.3" /> <!-- [kg] -->
     <xacro:property name="body_width" value="0.3" /> <!-- [m] -->

Commit message: all skins urdf

File: urdf/skin/link6_fancy.xacro (robot description, xacro)
@@ -1,9 +1,9 @@
 <?xml version="1.0"?>
-<robot name="link6" xmlns:xacro="http://ros.org/wiki/xacro">
+<robot xmlns:xacro="http://ros.org/wiki/xacro">
   <!-- Macro definition for link6 skin -->
   <xacro:macro name="link6_skin" params="parent namespace">
     <!-- Properties -->
     <xacro:property name="use_mesh_file" value="true" />
-    <xacro:property name="mesh_file" value="package://gentact_ros_tools/meshes/skin/link6_fancy.stl" />
+    <xacro:property name="mesh_file" value="package://gentact_ros_tools/meshes/skin/self-cap/link6_fancy.stl" />
     <xacro:property name="mass" value="0.3" /> <!-- [kg] -->
     <xacro:property name="body_width" value="0.3" /> <!-- [m] -->
