Commit message: compiled skin

File: urdf/skin/link6_big.xacro (robot description, xacro)
@@ -34,5 +34,5 @@
       normal_y="-0.771"
       normal_z="-0.155">
-      <origin xyz="-0.0831 -0.0491 -0.0215" rpy="1.726 0.000 -0.676" />
+      <origin xyz="-0.0631 -0.0491 -0.0215" rpy="1.726 0.000 -0.676" />
     </xacro:self_cap_sensor>
     <xacro:self_cap_sensor
@@ -45,5 +45,5 @@
       normal_y="-0.709"
       normal_z="0.702">
-      <origin xyz="-0.0553 -0.0490 0.0221" rpy="0.793 0.000 -0.103" />
+      <origin xyz="-0.0353 -0.0490 0.0221" rpy="0.793 0.000 -0.103" />
     </xacro:self_cap_sensor>
     <xacro:self_cap_sensor
@@ -56,5 +56,5 @@
       normal_y="-0.117"
       normal_z="0.014">
-      <origin xyz="0.0713 -0.0053 -0.0027" rpy="1.557 -0.000 1.454" />
+      <origin xyz="0.0913 -0.0053 -0.0027" rpy="1.557 -0.000 1.454" />
     </xacro:self_cap_sensor>
     <xacro:self_cap_sensor
@@ -67,5 +67,5 @@
       normal_y="-0.992"
       normal_z="0.008">
-      <origin xyz="-0.0122 -0.0561 -0.0028" rpy="1.563 -0.000 0.126" />
+      <origin xyz="0.0078 -0.0561 -0.0028" rpy="1.563 -0.000 0.126" />
     </xacro:self_cap_sensor>
     <xacro:self_cap_sensor
@@ -78,5 +78,5 @@
       normal_y="-0.960"
       normal_z="0.023">
-      <origin xyz="0.0375 -0.0444 -0.0024" rpy="1.548 -0.000 0.284" />
+      <origin xyz="0.0575 -0.0444 -0.0024" rpy="1.548 -0.000 0.284" />
     </xacro:self_cap_sensor>
     <xacro:self_cap_sensor
@@ -89,5 +89,5 @@
       normal_y="0.998"
       normal_z="0.042">
-      <origin xyz="0.0266 0.0474 0.0006" rpy="1.529 0.000 3.086" />
+      <origin xyz="0.0466 0.0474 0.0006" rpy="1.529 0.000 3.086" />
     </xacro:self_cap_sensor>
   </xacro:macro>
