Commit message: new xacro

File: urdf/robot/fr3_full_skin.xacro (robot description, xacro)
@@ -15,6 +15,6 @@
   <!-- <xacro:property name="link3_skin" value="package://gentact_ros_tools/urdf/skin/link3.xacro" /> -->
   <!-- <xacro:property name="link4_skin" value="package://gentact_ros_tools/urdf/skin/link4.xacro" /> -->
-  <xacro:property name="link5_skin" value="../skin/link5.xacro" />
-  <xacro:property name="link6_skin" value="../skin/link6.xacro" />
+  <xacro:property name="link5_skin" value="../skin/link5_fancy.xacro" />
+  <xacro:property name="link6_skin" value="../skin/link6_fancy.xacro" />
   <!-- <xacro:property name="link7_skin" value="package://gentact_ros_tools/urdf/skin/link7.xacro" /> -->
   <link name="base">

File: urdf/skin/link6_fancy.xacro (robot description, xacro)
@@ -5,5 +5,5 @@
     <!-- Properties -->
     <xacro:property name="use_mesh_file" value="true" />
-    <xacro:property name="mesh_file" value="package://gentact_ros_tools/meshes/skin/link6.stl" />
+    <xacro:property name="mesh_file" value="package://gentact_ros_tools/meshes/skin/link6_fancy.stl" />
     <xacro:property name="mass" value="0.3" /> <!-- [kg] -->
     <xacro:property name="body_width" value="0.3" /> <!-- [m] -->

Commit message: Reorganized

File: urdf/robot/fr3_full_skin.xacro (robot description, xacro)
@@ -11,11 +11,11 @@
   <!-- inertials: description of the inertials that comes from a YAML file. Example definition: ${xacro.load_yaml('$(find gentact_ros_tools)/robots/fr3/inertials.yaml')} -->
   <!-- dynamics: description of the dynamics that comes from a YAML file. Example definition: ${xacro.load_yaml('$(find gentact_ros_tools)/robots/fr3/dynamics.yaml')} -->
-  <!-- <xacro:property name="link1_skin" value="package://gentact_ros_tools/urdf/skin/link1.xacro" /> -->
-  <!-- <xacro:property name="link2_skin" value="package://gentact_ros_tools/urdf/skin/link2.xacro" /> -->
-  <!-- <xacro:property name="link3_skin" value="package://gentact_ros_tools/urdf/skin/link3.xacro" /> -->
-  <!-- <xacro:property name="link4_skin" value="package://gentact_ros_tools/urdf/skin/link4.xacro" /> -->
-  <xacro:property name="link5_skin" value="../skin/link5_fancy.xacro" />
-  <xacro:property name="link6_skin" value="../skin/link6_fancy.xacro" />
-  <!-- <xacro:property name="link7_skin" value="package://gentact_ros_tools/urdf/skin/link7.xacro" /> -->
+  <!-- Define arguments for skin configurations -->
+  <xacro:arg name="link1_skin" default=""/>
+  <xacro:arg name="link2_skin" default=""/>
+  <xacro:arg name="link3_skin" default=""/>
+  <xacro:arg name="link4_skin" default=""/>
+  <xacro:arg name="link5_skin" default=""/>
+  <xacro:arg name="link6_skin" default=""/>
   <link name="base">
       </link>
@@ -70,4 +70,10 @@
     <dynamics D="1" K="7000" damping="0.003" friction="0.2" mu_coulomb="0" mu_viscous="16"/>
   </joint>
+  <!-- Include the skin for link1 if specified -->
+  <xacro:property name="link1_skin_value" value="$(arg link1_skin)" />
+  <xacro:if value="${link1_skin_value != ''}">
+    <xacro:include filename="$(arg link1_skin)" />
+    <xacro:link1_skin parent="fr3_link1" namespace="link1" />
+  </xacro:if>
   <!-- sub-link defining detailed meshes for collision with environment -->
   <link name="fr3_link2">
@@ -97,4 +103,10 @@
     <dynamics D="1" K="7000" damping="0.003" friction="0.2" mu_coulomb="0" mu_viscous="16"/>
   </joint>
+  <!-- Include the skin for link2 if specified -->
+  <xacro:property name="link2_skin_value" value="$(arg link2_skin)" />
+  <xacro:if value="${link2_skin_value != ''}">
+    <xacro:include filename="$(arg link2_skin)" />
+    <xacro:link2_skin parent="fr3_link2" namespace="link2" />
+  </xacro:if>
   <!-- sub-link defining detailed meshes for collision with environment -->
   <link name="fr3_link3">
@@ -124,4 +136,10 @@
     <dynamics D="1" K="7000" damping="0.003" friction="0.2" mu_coulomb="0" mu_viscous="16"/>
   </joint>
+  <!-- Include the skin for link3 if specified -->
+  <xacro:property name="link3_skin_value" value="$(arg link3_skin)" />
+  <xacro:if value="${link3_skin_value != ''}">
+    <xacro:include filename="$(arg link3_skin)" />
+    <xacro:link3_skin parent="fr3_link3" namespace="link3" />
+  </xacro:if>
   <!-- sub-link defining detailed meshes for collision with environment -->
   <link name="fr3_link4">
@@ -151,4 +169,10 @@
     <dynamics D="1" K="7000" damping="0.003" friction="0.2" mu_coulomb="0" mu_viscous="16"/>
   </joint>
+  <!-- Include the skin for link4 if specified -->
+  <xacro:property name="link4_skin_value" value="$(arg link4_skin)" />
+  <xacro:if value="${link4_skin_value != ''}">
+    <xacro:include filename="$(arg link4_skin)" />
+    <xacro:link4_skin parent="fr3_link4" namespace="link4" />
+  </xacro:if>
   <!-- sub-link defining detailed meshes for collision with environment -->
   <link name="fr3_link5">
@@ -178,7 +202,10 @@
     <dynamics D="1" K="7000" damping="0.003" friction="0.2" mu_coulomb="0" mu_viscous="16"/>
   </joint>
-  <!-- Include the skin for link5 -->
-  <xacro:include filename="${link5_skin}" />
-  <xacro:link5_skin parent="fr3_link5" namespace="link5" />
+  <!-- Include the skin for link5 if specified -->
+  <xacro:property name="link5_skin_value" value="$(arg link5_skin)" />
+  <xacro:if value="${link5_skin_value != ''}">
+    <xacro:include filename="$(arg link5_skin)" />
+    <xacro:link5_skin parent="fr3_link5" namespace="link5" />
+  </xacro:if>
   <!-- sub-link defining detailed meshes for collision with environment -->
   <link name="fr3_link6">
@@ -208,7 +235,10 @@
     <dynamics D="1" K="7000" damping="0.003" friction="0.2" mu_coulomb="0" mu_viscous="16"/>
   </joint>
-  <!-- Include the skin for link6 -->
-  <xacro:include filename="${link6_skin}" />
-  <xacro:link6_skin parent="fr3_link6" namespace="link6" />
+  <!-- Include the skin for link6 if specified -->
+  <xacro:property name="link6_skin_value" value="$(arg link6_skin)" />
+  <xacro:if value="${link6_skin_value != ''}">
+    <xacro:include filename="$(arg link6_skin)" />
+    <xacro:link6_skin parent="fr3_link6" namespace="link6" />
+  </xacro:if>
   <!-- sub-link defining detailed meshes for collision with environment -->
   <link name="fr3_link7">
@@ -244,131 +274,3 @@
     <child link="fr3_link8"/>
   </joint>
-  <joint name="fr3_hand_joint" type="fixed">
-    <parent link="fr3_link8"/>
-    <child link="fr3_hand"/>
-    <origin rpy="0 0 -0.7853981633974483" xyz="0 0 0"/>
-  </joint>
-  <!-- sub-link defining detailed meshes for collision with environment -->
-  <link name="fr3_hand">
-    <visual name="fr3_hand_visual">
-      <geometry>
-        <mesh filename="package://gentact_ros_tools/meshes/robot_ee/franka_hand_white/visual/hand.dae"/>
-      </geometry>
-    </visual>
-    <collision name="fr3_hand_collision">
-      <geometry>
-        <mesh filename="package://gentact_ros_tools/meshes/robot_ee/franka_hand_white/collision/hand.stl"/>
-      </geometry>
-    </collision>
-    <inertial>
-      <origin rpy="0 0 0" xyz="-0.0000376 0.0119128 0.0207260"/>
-      <mass value="0.6544"/>
-      <inertia ixx="0.00186" ixy="0.0" ixz="0.0" iyy="0.0003" iyz="-2e-05" izz="0.00174"/>
-    </inertial>
-  </link>
-  <!-- Define the hand_tcp frame -->
-  <link name="fr3_hand_tcp"/>
-  <joint name="fr3_hand_tcp_joint" type="fixed">
-    <origin rpy="0 0 0" xyz="0 0 0.1034"/>
-    <parent link="fr3_hand"/>
-    <child link="fr3_hand_tcp"/>
-  </joint>
-  <link name="fr3_leftfinger">
-    <visual name="fr3_leftfinger_visual">
-      <geometry>
-        <mesh filename="package://gentact_ros_tools/meshes/robot_ee/franka_hand_white/visual/finger.dae"/>
-      </geometry>
-    </visual>
-    <!-- screw mount -->
-    <collision>
-      <origin rpy="0 0 0" xyz="0 18.5e-3 11e-3"/>
-      <geometry>
-        <box size="22e-3 15e-3 20e-3"/>
-      </geometry>
-    </collision>
-    <!-- cartriage sledge -->
-    <collision>
-      <origin rpy="0 0 0" xyz="0 6.8e-3 2.2e-3"/>
-      <geometry>
-        <box size="22e-3 8.8e-3 3.8e-3"/>
-      </geometry>
-    </collision>
-    <!-- diagonal finger -->
-    <collision>
-      <origin rpy="0.5235987755982988 0 0" xyz="0 15.9e-3 28.35e-3"/>
-      <geometry>
-        <box size="17.5e-3 7e-3 23.5e-3"/>
-      </geometry>
-    </collision>
-    <!-- rubber tip with which to grasp -->
-    <collision>
-      <origin rpy="0 0 0" xyz="0 7.58e-3 45.25e-3"/>
-      <geometry>
-        <box size="17.5e-3 15.2e-3 18.5e-3"/>
-      </geometry>
-    </collision>
-    <inertial>
-      <origin rpy="0 0 0" xyz="0 0.0152850 0.0219675"/>
-      <mass value="0.0291"/>
-      <inertia ixx="8.49e-06" ixy="0.0" ixz="0.0" iyy="8.53e-06" iyz="-1.06e-06" izz="1.77e-06"/>
-    </inertial>
-  </link>
-  <link name="fr3_rightfinger">
-    <visual name="fr3_rightfinger_visual">
-      <origin rpy="0 0 0" xyz="0 0 0"/>
-      <geometry>
-        <mesh filename="package://gentact_ros_tools/meshes/robot_ee/franka_hand_white/visual/finger.dae"/>
-      </geometry>
-    </visual>
-    <!-- screw mount -->
-    <collision>
-      <origin rpy="0 0 0" xyz="0 18.5e-3 11e-3"/>
-      <geometry>
-        <box size="22e-3 15e-3 20e-3"/>
-      </geometry>
-    </collision>
-    <!-- cartriage sledge -->
-    <collision>
-      <origin rpy="0 0 0" xyz="0 6.8e-3 2.2e-3"/>
-      <geometry>
-        <box size="22e-3 8.8e-3 3.8e-3"/>
-      </geometry>
-    </collision>
-    <!-- diagonal finger -->
-    <collision>
-      <origin rpy="-0.5235987755982988 0 3.141592653589793" xyz="0 15.9e-3 28.35e-3"/>
-      <geometry>
-        <box size="17.5e-3 7e-3 23.5e-3"/>
-      </geometry>
-    </collision>
-    <!-- rubber tip with which to grasp -->
-    <collision>
-      <origin rpy="0 0 0" xyz="0 7.58e-3 45.25e-3"/>
-      <geometry>
-        <box size="17.5e-3 15.2e-3 18.5e-3"/>
-      </geometry>
-    </collision>
-    <inertial>
-      <origin rpy="0 0 0" xyz="0 0.0152850 0.0219675"/>
-      <mass value="0.0291"/>
-      <inertia ixx="8.49e-06" ixy="0.0" ixz="0.0" iyy="8.53e-06" iyz="-1.06e-06" izz="1.77e-06"/>
-    </inertial>
-  </link>
-  <joint name="fr3_finger_joint1" type="prismatic">
-    <parent link="fr3_hand"/>
-    <child link="fr3_leftfinger"/>
-    <origin rpy="0 0 0" xyz="0 0 0.0584"/>
-    <axis xyz="0 1 0"/>
-    <limit effort="100" lower="0.0" upper="0.04" velocity="0.2"/>
-    <dynamics damping="0.3"/>
-  </joint>
-  <joint name="fr3_finger_joint2" type="prismatic">
-    <parent link="fr3_hand"/>
-    <child link="fr3_rightfinger"/>
-    <origin rpy="0 0 3.141592653589793" xyz="0 0 0.0584"/>
-    <axis xyz="0 1 0"/>
-    <limit effort="100" lower="0.0" upper="0.04" velocity="0.2"/>
-    <mimic joint="fr3_finger_joint1"/>
-    <dynamics damping="0.3"/>
-  </joint>
 </robot>

File: urdf/skin/link5_fancy.xacro (robot description, xacro)
@@ -22,87 +22,72 @@
       use_mesh_file="${use_mesh_file}"
       mesh_file="${mesh_file}">
-      <inertial>
-        <mass value="${mass}" />
-        <origin xyz="0 0 0" rpy="0 0 0" />
-        <inertia ixx="0.001" ixy="0.0" ixz="0.0" iyy="0.001" iyz="0.0" izz="0.001" />
-      </inertial>
+      <origin xyz="0 0 0" rpy="0 0 0" />
     </xacro:dermis_base_macro>
     <!-- Instantiate sensors -->
     <xacro:self_cap_sensor
       robot_namespace="${namespace}"
-      parent="${namespace}/base_link"
+      parent="${namespace}_skin"
       sensor_number="0"
       sensor_radius="${sensor_radius}"
       sensor_length="0.057"
-      normal_x="-0.465"
-      normal_y="-0.066"
-      normal_z="0.883">
-      <origin xyz="-0.032 -0.092 0.057" rpy="0.488 0.000 -1.431" />
+      normal_x="-0.049"
+      normal_y="0.985"
+      normal_z="-0.167">
+      <origin xyz="-0.004 0.115 -0.089" rpy="-1.403 -3.142 0.049" />
     </xacro:self_cap_sensor>
     <xacro:self_cap_sensor
       robot_namespace="${namespace}"
-      parent="${namespace}/base_link"
+      parent="${namespace}_skin"
       sensor_number="1"
       sensor_radius="${sensor_radius}"
       sensor_length="0.048"
-      normal_x="-0.120"
-      normal_y="-0.740"
-      normal_z="0.661">
-      <origin xyz="-0.007 -0.131 0.048" rpy="0.848 0.000 -0.160" />
+      normal_x="-0.050"
+      normal_y="0.941"
+      normal_z="-0.335">
+      <origin xyz="-0.007 0.127 -0.038" rpy="-1.229 -3.142 0.054" />
     </xacro:self_cap_sensor>
     <xacro:self_cap_sensor
       robot_namespace="${namespace}"
-      parent="${namespace}/base_link"
+      parent="${namespace}_skin"
       sensor_number="2"
       sensor_radius="${sensor_radius}"
       sensor_length="0.060"
-      normal_x="0.276"
-      normal_y="0.006"
-      normal_z="0.961">
-      <origin xyz="0.023 -0.086 0.060" rpy="0.280 -0.000 1.591" />
+      normal_x="0.375"
+      normal_y="0.908"
+      normal_z="-0.188">
+      <origin xyz="0.026 0.130 -0.013" rpy="1.760 -0.000 2.750" />
     </xacro:self_cap_sensor>
     <xacro:self_cap_sensor
       robot_namespace="${namespace}"
-      parent="${namespace}/base_link"
+      parent="${namespace}_skin"
       sensor_number="3"
       sensor_radius="${sensor_radius}"
       sensor_length="0.059"
-      normal_x="-0.021"
-      normal_y="0.008"
-      normal_z="1.000">
-      <origin xyz="-0.002 -0.034 0.059" rpy="0.023 0.000 -1.950" />
+      normal_x="-0.230"
+      normal_y="0.956"
+      normal_z="-0.183">
+      <origin xyz="-0.016 0.104 -0.138" rpy="1.754 0.000 -2.906" />
     </xacro:self_cap_sensor>
     <xacro:self_cap_sensor
       robot_namespace="${namespace}"
-      parent="${namespace}/base_link"
+      parent="${namespace}_skin"
       sensor_number="4"
       sensor_radius="${sensor_radius}"
       sensor_length="0.059"
-      normal_x="-0.333"
-      normal_y="-0.001"
-      normal_z="0.943">
-      <origin xyz="-0.020 0.060 0.059" rpy="0.339 -0.000 -1.569" />
+      normal_x="-0.092"
+      normal_y="0.902"
+      normal_z="0.422">
+      <origin xyz="-0.007 0.133 0.023" rpy="1.136 0.000 -3.040" />
     </xacro:self_cap_sensor>
     <xacro:self_cap_sensor
       robot_namespace="${namespace}"
-      parent="${namespace}/base_link"
+      parent="${namespace}_skin"
       sensor_number="5"
       sensor_radius="${sensor_radius}"
       sensor_length="0.025"
-      normal_x="0.845"
-      normal_y="-0.481"
-      normal_z="0.235">
-      <origin xyz="0.049 -0.115 0.025" rpy="1.334 0.000 1.053" />
-    </xacro:self_cap_sensor>
-    <xacro:self_cap_sensor
-      robot_namespace="${namespace}"
-      parent="${namespace}/base_link"
-      sensor_number="6"
-      sensor_radius="${sensor_radius}"
-      sensor_length="0.023"
-      normal_x="-0.845"
-      normal_y="-0.475"
-      normal_z="0.246">
-      <origin xyz="-0.049 -0.116 0.023" rpy="1.323 0.000 -1.059" />
+      normal_x="-0.018"
+      normal_y="0.953"
+      normal_z="-0.304">
+      <origin xyz="-0.000 0.096 -0.184" rpy="-1.262 3.142 0.019" />
     </xacro:self_cap_sensor>
   </xacro:macro>

File: urdf/skin/link6_fancy.xacro (robot description, xacro)
@@ -22,9 +22,5 @@
       use_mesh_file="${use_mesh_file}"
       mesh_file="${mesh_file}">
-      <inertial>
-        <mass value="${mass}" />
-        <origin xyz="0 0 0" rpy="0 0 0" />
-        <inertia ixx="0.001" ixy="0.0" ixz="0.0" iyy="0.001" iyz="0.0" izz="0.001" />
-      </inertial>
+      <origin xyz="0 0 0" rpy="-1.57079632679 0 0" />
     </xacro:dermis_base_macro>
     <!-- Instantiate sensors -->

File: urdf/skin/self-cap-base.xacro (robot description, xacro)
@@ -3,11 +3,5 @@
   <!-- Main Sensor Dermis -->
   <xacro:macro name="dermis_base_macro"
-    params="robot_namespace parent mass body_width body_height use_mesh_file mesh_file *inertia">
-    <link name="${robot_namespace}_skin"></link>
-    <joint name="${robot_namespace}_base_joint" type="fixed">
-      <origin xyz="0 0 0" rpy="0 0 0" />
-      <parent link="${parent}" />
-      <child link="${robot_namespace}_skin" />
-    </joint>
+    params="robot_namespace parent mass body_width body_height use_mesh_file mesh_file *origin">
     <link name="${robot_namespace}_skin">
       <visual>
@@ -23,4 +17,9 @@
       </visual>
     </link>
+    <joint name="${robot_namespace}_base_joint" type="fixed">
+      <xacro:insert_block name="origin" />
+      <parent link="${parent}" />
+      <child link="${robot_namespace}_skin" />
+    </joint>
   </xacro:macro>
   <!-- Self Capacitance Proximity Sensor -->

Commit message: Calibration script

File: urdf/robot/fr3_full_skin.xacro (robot description, xacro)
@@ -18,4 +18,5 @@
   <xacro:arg name="link5_skin" default=""/>
   <xacro:arg name="link6_skin" default=""/>
+  <xacro:arg name="ee_xacro_file" default=""/>
   <link name="base">
       </link>
@@ -268,9 +269,10 @@
     <dynamics D="1" K="7000" damping="0.003" friction="0.2" mu_coulomb="0" mu_viscous="16"/>
   </joint>
-  <link name="fr3_link8"/>
-  <joint name="fr3_joint8" type="fixed">
-    <origin rpy="0 0 0" xyz="0 0 0.107"/>
-    <parent link="fr3_link7"/>
-    <child link="fr3_link8"/>
-  </joint>
+  <!-- End effector -->
+  <!-- Include the end effector if specified -->
+  <xacro:property name="ee_xacro_file" value="$(arg ee_xacro_file)" />
+  <xacro:if value="${ee_xacro_file != ''}">
+    <xacro:include filename="$(arg ee_xacro_file)" />
+    <xacro:ee_macro parent="fr3_link7"/>
+  </xacro:if>
 </robot>
