Commit message: Finished data collection

File: urdf/calibration/link4.xacro (robot description, xacro)
@@ -1,9 +1,9 @@
 <?xml version="1.0"?>
 <robot name="calibration_skin" xmlns:xacro="http://ros.org/wiki/xacro">
-  <!-- Include the link5 skin macro -->
+  <!-- Include the link4 skin macro -->
   <xacro:include filename="$(find gentact_ros_tools)/urdf/skin/link4_fancy.xacro" />
   <!-- Create a base link for the calibration skin -->
   <link name="calibration_base" />
-  <!-- Instantiate the link5 skin -->
+  <!-- Instantiate the link4 skin -->
   <xacro:link4_skin
     parent="calibration_base"

File: urdf/skin/link2_fancy.xacro (robot description, xacro)
@@ -28,5 +28,5 @@
       robot_namespace="${namespace}"
       parent="${namespace}_skin"
-      sensor_number="0"
+      sensor_number="3"
       sensor_radius="${sensor_radius}"
       sensor_length="0.05"
@@ -39,5 +39,5 @@
       robot_namespace="${namespace}"
       parent="${namespace}_skin"
-      sensor_number="1"
+      sensor_number="2"
       sensor_radius="${sensor_radius}"
       sensor_length="0.05"
@@ -50,5 +50,5 @@
       robot_namespace="${namespace}"
       parent="${namespace}_skin"
-      sensor_number="2"
+      sensor_number="0"
       sensor_radius="${sensor_radius}"
       sensor_length="0.05"
@@ -61,5 +61,5 @@
       robot_namespace="${namespace}"
       parent="${namespace}_skin"
-      sensor_number="3"
+      sensor_number="6"
       sensor_radius="${sensor_radius}"
       sensor_length="0.05"
@@ -72,5 +72,5 @@
       robot_namespace="${namespace}"
       parent="${namespace}_skin"
-      sensor_number="4"
+      sensor_number="1"
       sensor_radius="${sensor_radius}"
       sensor_length="0.05"
@@ -94,5 +94,5 @@
       robot_namespace="${namespace}"
       parent="${namespace}_skin"
-      sensor_number="6"
+      sensor_number="4"
       sensor_radius="${sensor_radius}"
       sensor_length="0.05"

File: urdf/skin/link3_fancy.xacro (robot description, xacro)
@@ -39,5 +39,5 @@
       robot_namespace="${namespace}"
       parent="${namespace}_skin"
-      sensor_number="6"
+      sensor_number="2"
       sensor_radius="${sensor_radius}"
       sensor_length="0.05"
@@ -50,5 +50,5 @@
       robot_namespace="${namespace}"
       parent="${namespace}_skin"
-      sensor_number="0"
+      sensor_number="1"
       sensor_radius="${sensor_radius}"
       sensor_length="0.05"
@@ -72,5 +72,5 @@
       robot_namespace="${namespace}"
       parent="${namespace}_skin"
-      sensor_number="4"
+      sensor_number="6"
       sensor_radius="${sensor_radius}"
       sensor_length="0.05"
@@ -83,5 +83,5 @@
       robot_namespace="${namespace}"
       parent="${namespace}_skin"
-      sensor_number="3"
+      sensor_number="4"
       sensor_radius="${sensor_radius}"
       sensor_length="0.05"
@@ -94,5 +94,5 @@
       robot_namespace="${namespace}"
       parent="${namespace}_skin"
-      sensor_number="1"
+      sensor_number="0"
       sensor_radius="${sensor_radius}"
       sensor_length="0.05"
@@ -105,5 +105,5 @@
       robot_namespace="${namespace}"
       parent="${namespace}_skin"
-      sensor_number="2"
+      sensor_number="3"
       sensor_radius="${sensor_radius}"
       sensor_length="0.05"

File: urdf/skin/link4_fancy.xacro (robot description, xacro)
@@ -1,9 +1,9 @@
 <?xml version="1.0"?>
 <robot xmlns:xacro="http://ros.org/wiki/xacro">
-  <!-- Macro definition for link1 skin -->
-  <xacro:macro name="link1_skin" params="parent namespace">
+  <!-- Macro definition for link4 skin -->
+  <xacro:macro name="link4_skin" params="parent namespace">
     <!-- Properties -->
     <xacro:property name="use_mesh_file" value="true" />
-    <xacro:property name="mesh_file" value="package://gentact_ros_tools/meshes/skin/self-cap/link1_fancy.stl" />
+    <xacro:property name="mesh_file" value="package://gentact_ros_tools/meshes/skin/self-cap/link4_fancy.stl" />
     <xacro:property name="mass" value="0.3" /> <!-- [kg] -->
     <xacro:property name="body_width" value="0.3" /> <!-- [m] -->
@@ -31,8 +31,30 @@
       sensor_radius="${sensor_radius}"
       sensor_length="0.05"
-      normal_x="-0.864"
-      normal_y="-0.453"
-      normal_z="0.219">
-      <origin xyz="-0.050 -0.111 0.013" rpy="1.350 0.000 -1.088" />
+      normal_x="-0.053"
+      normal_y="-0.985"
+      normal_z="-0.165">
+      <origin xyz="-0.075 -0.054 0.047" rpy="1.737 -0.000 -0.054" />
+    </xacro:self_cap_sensor>
+    <xacro:self_cap_sensor
+      robot_namespace="${namespace}"
+      parent="${namespace}_skin"
+      sensor_number="4"
+      sensor_radius="${sensor_radius}"
+      sensor_length="0.05"
+      normal_x="-0.486"
+      normal_y="0.868"
+      normal_z="-0.103">
+      <origin xyz="-0.112 0.052 0.084" rpy="1.674 -0.000 -2.632" />
+    </xacro:self_cap_sensor>
+    <xacro:self_cap_sensor
+      robot_namespace="${namespace}"
+      parent="${namespace}_skin"
+      sensor_number="5"
+      sensor_radius="${sensor_radius}"
+      sensor_length="0.05"
+      normal_x="0.622"
+      normal_y="-0.345"
+      normal_z="0.703">
+      <origin xyz="0.034 -0.088 0.038" rpy="0.791 -0.000 1.064" />
     </xacro:self_cap_sensor>
     <xacro:self_cap_sensor
@@ -42,8 +64,8 @@
       sensor_radius="${sensor_radius}"
       sensor_length="0.05"
-      normal_x="-0.560"
-      normal_y="-0.826"
-      normal_z="-0.067">
-      <origin xyz="-0.034 -0.053 -0.135" rpy="1.638 0.000 -0.596" />
+      normal_x="-0.689"
+      normal_y="-0.719"
+      normal_z="-0.086">
+      <origin xyz="-0.044 -0.101 -0.003" rpy="1.657 0.000 -0.764" />
     </xacro:self_cap_sensor>
     <xacro:self_cap_sensor
@@ -53,8 +75,8 @@
       sensor_radius="${sensor_radius}"
       sensor_length="0.05"
-      normal_x="0.309"
-      normal_y="-0.948"
-      normal_z="-0.082">
-      <origin xyz="0.019 -0.060 -0.138" rpy="1.653 -0.000 0.315" />
+      normal_x="-0.358"
+      normal_y="-0.243"
+      normal_z="0.901">
+      <origin xyz="-0.024 -0.076 0.049" rpy="0.448 0.000 -0.975" />
     </xacro:self_cap_sensor>
     <xacro:self_cap_sensor
@@ -64,52 +86,8 @@
       sensor_radius="${sensor_radius}"
       sensor_length="0.05"
-      normal_x="-0.374"
-      normal_y="-0.638"
-      normal_z="-0.673">
-      <origin xyz="-0.023 -0.113 -0.044" rpy="2.309 0.000 -0.530" />
-    </xacro:self_cap_sensor>
-    <xacro:self_cap_sensor
-      robot_namespace="${namespace}"
-      parent="${namespace}_skin"
-      sensor_number="4"
-      sensor_radius="${sensor_radius}"
-      sensor_length="0.05"
-      normal_x="0.378"
-      normal_y="-0.800"
-      normal_z="-0.467">
-      <origin xyz="0.023 -0.074 -0.084" rpy="2.057 0.000 0.441" />
-    </xacro:self_cap_sensor>
-    <xacro:self_cap_sensor
-      robot_namespace="${namespace}"
-      parent="${namespace}_skin"
-      sensor_number="5"
-      sensor_radius="${sensor_radius}"
-      sensor_length="0.05"
-      normal_x="0.845"
-      normal_y="-0.486"
-      normal_z="0.223">
-      <origin xyz="0.049 -0.112 0.012" rpy="1.346 -0.000 1.049" />
-    </xacro:self_cap_sensor>
-    <xacro:self_cap_sensor
-      robot_namespace="${namespace}"
-      parent="${namespace}_skin"
-      sensor_number="6"
-      sensor_radius="${sensor_radius}"
-      sensor_length="0.05"
-      normal_x="-0.086"
-      normal_y="-0.992"
-      normal_z="0.094">
-      <origin xyz="-0.006 -0.136 0.006" rpy="1.477 0.000 -0.087" />
-    </xacro:self_cap_sensor>
-    <xacro:self_cap_sensor
-      robot_namespace="${namespace}"
-      parent="${namespace}_skin"
-      sensor_number="7"
-      sensor_radius="${sensor_radius}"
-      sensor_length="0.05"
-      normal_x="0.497"
-      normal_y="-0.590"
-      normal_z="-0.636">
-      <origin xyz="0.030 -0.112 -0.041" rpy="2.260 0.000 0.700" />
+      normal_x="0.148"
+      normal_y="-0.982"
+      normal_z="-0.117">
+      <origin xyz="0.010 -0.117 -0.008" rpy="1.688 -0.000 0.150" />
     </xacro:self_cap_sensor>
   </xacro:macro>

File: urdf/skin/link6_fancy.xacro (robot description, xacro)
@@ -28,5 +28,5 @@
       robot_namespace="${namespace}"
       parent="${namespace}_skin"
-      sensor_number="0"
+      sensor_number="2"
       sensor_radius="${sensor_radius}"
       sensor_length="0.057"
@@ -39,5 +39,5 @@
       robot_namespace="${namespace}"
       parent="${namespace}_skin"
-      sensor_number="1"
+      sensor_number="0"
       sensor_radius="${sensor_radius}"
       sensor_length="0.048"
@@ -50,5 +50,5 @@
       robot_namespace="${namespace}"
       parent="${namespace}_skin"
-      sensor_number="2"
+      sensor_number="3"
       sensor_radius="${sensor_radius}"
       sensor_length="0.060"
@@ -61,5 +61,5 @@
       robot_namespace="${namespace}"
       parent="${namespace}_skin"
-      sensor_number="3"
+      sensor_number="6"
       sensor_radius="${sensor_radius}"
       sensor_length="0.059"
@@ -72,5 +72,5 @@
       robot_namespace="${namespace}"
       parent="${namespace}_skin"
-      sensor_number="4"
+      sensor_number="5"
       sensor_radius="${sensor_radius}"
       sensor_length="0.059"
@@ -83,5 +83,5 @@
       robot_namespace="${namespace}"
       parent="${namespace}_skin"
-      sensor_number="5"
+      sensor_number="4"
       sensor_radius="${sensor_radius}"
       sensor_length="0.025"
@@ -94,5 +94,5 @@
       robot_namespace="${namespace}"
       parent="${namespace}_skin"
-      sensor_number="6"
+      sensor_number="1"
       sensor_radius="${sensor_radius}"
       sensor_length="0.023"
