Commit message: add link2 correct orientation

File: meshes/skin/hybrid/link1_hybrid.xacro (robot description, xacro)
@@ -5,5 +5,5 @@
     <!-- Properties -->
     <xacro:property name="use_mesh_file" value="true" />
-    <xacro:property name="mesh_file" value="package://gentact_descriptions_hybrid/meshes/skin/hybrid/link2_hybrid_dermis.stl" />
+    <xacro:property name="mesh_file" value="package://gentact_descriptions_hybrid/meshes/skin/hybrid/link1_hybrid_dermis.stl" />
     <xacro:property name="mass" value="0.3" /> <!-- [kg] -->
     <xacro:property name="body_width" value="0.3" /> <!-- [m] -->
@@ -22,35 +22,34 @@
       use_mesh_file="${use_mesh_file}"
       mesh_file="${mesh_file}">
-      <origin xyz="0 0 0" rpy="-1.5707 0 0" />
+      <origin xyz="0 0 0" rpy="3.14159265359 0 0" />
     </xacro:dermis_base_macro>
-    <!-- Instantiate sensors -->
     <xacro:self_cap_sensor robot_namespace="${namespace}" parent="${namespace}_skin" sensor_number="0"
+      sensor_radius="${sensor_radius}" sensor_length="${sensor_length}" normal_x="0.106" normal_y="0.989" normal_z="-0.108">
+      <origin xyz="0.007 0.136 -0.007" rpy="-1.463 -3.142 -0.106" />
+    </xacro:self_cap_sensor>
+    <xacro:self_cap_sensor robot_namespace="${namespace}" parent="${namespace}_skin" sensor_number="1"
+      sensor_radius="${sensor_radius}" sensor_length="${sensor_length}" normal_x="-0.341" normal_y="0.683" normal_z="0.646">
+      <origin xyz="-0.024 0.113 0.045" rpy="0.869 -0.000 -2.678" />
+    </xacro:self_cap_sensor>
+    <xacro:self_cap_sensor robot_namespace="${namespace}" parent="${namespace}_skin" sensor_number="2"
+      sensor_radius="${sensor_radius}" sensor_length="${sensor_length}" normal_x="-0.777" normal_y="0.627" normal_z="-0.060">
+      <origin xyz="-0.050 0.113 -0.009" rpy="1.630 -0.000 -2.249" />
+    </xacro:self_cap_sensor>
+    <xacro:self_cap_sensor robot_namespace="${namespace}" parent="${namespace}_skin" sensor_number="3"
       sensor_radius="${sensor_radius}" sensor_length="${sensor_length}" normal_x="0.723" normal_y="0.688" normal_z="-0.056">
       <origin xyz="0.052 0.111 -0.004" rpy="1.627 -0.000 2.332" />
     </xacro:self_cap_sensor>
-    <xacro:self_cap_sensor robot_namespace="${namespace}" parent="${namespace}_skin" sensor_number="1"
+    <xacro:self_cap_sensor robot_namespace="${namespace}" parent="${namespace}_skin" sensor_number="4"
       sensor_radius="${sensor_radius}" sensor_length="${sensor_length}" normal_x="0.458" normal_y="0.631" normal_z="0.627">
       <origin xyz="0.029 0.112 0.042" rpy="0.893 0.000 2.514" />
     </xacro:self_cap_sensor>
-    <xacro:self_cap_sensor robot_namespace="${namespace}" parent="${namespace}_skin" sensor_number="2"
-      sensor_radius="${sensor_radius}" sensor_length="${sensor_length}" normal_x="0.106" normal_y="0.989" normal_z="-0.108">
-      <origin xyz="0.007 0.136 -0.007" rpy="-1.463 -3.142 -0.106" />
-    </xacro:self_cap_sensor>
-    <xacro:self_cap_sensor robot_namespace="${namespace}" parent="${namespace}_skin" sensor_number="3"
+    <xacro:self_cap_sensor robot_namespace="${namespace}" parent="${namespace}_skin" sensor_number="5"
       sensor_radius="${sensor_radius}" sensor_length="${sensor_length}" normal_x="0.222" normal_y="0.969" normal_z="0.105">
       <origin xyz="0.009 0.064 0.131" rpy="1.466 0.000 2.917" />
     </xacro:self_cap_sensor>
-    <xacro:self_cap_sensor robot_namespace="${namespace}" parent="${namespace}_skin" sensor_number="4"
+    <xacro:self_cap_sensor robot_namespace="${namespace}" parent="${namespace}_skin" sensor_number="6"
       sensor_radius="${sensor_radius}" sensor_length="${sensor_length}" normal_x="-0.133" normal_y="0.605" normal_z="-0.785">
       <origin xyz="-0.009 0.112 -0.051" rpy="-0.668 -3.142 0.217" />
     </xacro:self_cap_sensor>
-    <xacro:self_cap_sensor robot_namespace="${namespace}" parent="${namespace}_skin" sensor_number="5"
-      sensor_radius="${sensor_radius}" sensor_length="${sensor_length}" normal_x="-0.341" normal_y="0.683" normal_z="0.646">
-      <origin xyz="-0.024 0.113 0.045" rpy="0.869 -0.000 -2.678" />
-    </xacro:self_cap_sensor>
-    <xacro:self_cap_sensor robot_namespace="${namespace}" parent="${namespace}_skin" sensor_number="6"
-      sensor_radius="${sensor_radius}" sensor_length="${sensor_length}" normal_x="-0.777" normal_y="0.627" normal_z="-0.060">
-      <origin xyz="-0.050 0.113 -0.009" rpy="1.630 -0.000 -2.249" />
-    </xacro:self_cap_sensor>
   </xacro:macro>
      </robot>

File: meshes/skin/hybrid/link3_hybrid.xacro (robot description, xacro)
@@ -5,5 +5,5 @@
     <!-- Properties -->
     <xacro:property name="use_mesh_file" value="true" />
-    <xacro:property name="mesh_file" value="package://gentact_descriptions/meshes/skin/hybrid/link3_hybrid_dermis.stl" />
+    <xacro:property name="mesh_file" value="package://gentact_descriptions_hybrid/meshes/skin/hybrid/link3_hybrid_dermis.stl" />
     <xacro:property name="mass" value="0.3" /> <!-- [kg] -->
     <xacro:property name="body_width" value="0.3" /> <!-- [m] -->
@@ -12,5 +12,5 @@
     <xacro:property name="sensor_radius" value="0.0" /> <!-- [m] -->
     <!-- Included URDF Files -->
-    <xacro:include filename="$(find gentact_descriptions)/robots/common/skin_unit_base.xacro" />
+    <xacro:include filename="$(find gentact_descriptions_hybrid)/robots/common/skin_unit_base.xacro" />
     <!-- Instantiate dermis once -->
     <xacro:dermis_base_macro

File: meshes/skin/hybrid/link4_hybrid.xacro (robot description, xacro)
@@ -5,5 +5,5 @@
     <!-- Properties -->
     <xacro:property name="use_mesh_file" value="true" />
-    <xacro:property name="mesh_file" value="package://gentact_descriptions/meshes/skin/hybrid/link4_hybrid_dermis.stl" />
+    <xacro:property name="mesh_file" value="package://gentact_descriptions_hybrid/meshes/skin/hybrid/link4_hybrid_dermis.stl" />
     <xacro:property name="mass" value="0.3" /> <!-- [kg] -->
     <xacro:property name="body_width" value="0.3" /> <!-- [m] -->
@@ -12,5 +12,5 @@
     <xacro:property name="sensor_radius" value="0.0" /> <!-- [m] -->
     <!-- Included URDF Files -->
-    <xacro:include filename="$(find gentact_ros_tools)/urdf/skin/self-cap-base.xacro" />
+    <xacro:include filename="$(find gentact_ros_tools_hybrid)/urdf/skin/self-cap-base.xacro" />
     <!-- Instantiate dermis once -->
     <xacro:dermis_base_macro

File: meshes/skin/hybrid/link5_hybrid.xacro (robot description, xacro)
@@ -5,5 +5,5 @@
     <!-- Properties -->
     <xacro:property name="use_mesh_file" value="true" />
-    <xacro:property name="mesh_file" value="package://gentact_ros_tools/meshes/skin/hybrid/link5_hybrid_dermis.stl" />
+    <xacro:property name="mesh_file" value="package://gentact_ros_tools_hybrid/meshes/skin/hybrid/link5_hybrid_dermis.stl" />
     <xacro:property name="mass" value="0.3" /> <!-- [kg] -->
     <xacro:property name="body_width" value="0.3" /> <!-- [m] -->
@@ -12,5 +12,5 @@
     <xacro:property name="sensor_radius" value="0.0" /> <!-- [m] -->
     <!-- Included URDF Files -->
-    <xacro:include filename="$(find gentact_ros_tools)/urdf/skin/self-cap-base.xacro" />
+    <xacro:include filename="$(find gentact_ros_tools_hybrid)/urdf/skin/self-cap-base.xacro" />
     <!-- Instantiate dermis once -->
     <xacro:dermis_base_macro

File: meshes/skin/hybrid/link5_hybrid_back.xacro (robot description, xacro)
@@ -5,5 +5,5 @@
     <!-- Properties -->
     <xacro:property name="use_mesh_file" value="true" />
-    <xacro:property name="mesh_file" value="package://gentact_descriptions/meshes/skin/hybrid/link5_part2_hybrid_dermis.stl" />
+    <xacro:property name="mesh_file" value="package://gentact_descriptions_hybrid/meshes/skin/hybrid/link5_part2_hybrid_dermis.stl" />
     <xacro:property name="mass" value="0.3" /> <!-- [kg] -->
     <xacro:property name="body_width" value="0.3" /> <!-- [m] -->
@@ -12,5 +12,5 @@
     <xacro:property name="sensor_radius" value="0.0" /> <!-- [m] -->
     <!-- Included URDF Files -->
-    <xacro:include filename="$(find gentact_ros_tools)/urdf/skin/self-cap-base.xacro" />
+    <xacro:include filename="$(find gentact_ros_tools_hybrid)/urdf/skin/self-cap-base.xacro" />
     <!-- Instantiate dermis once -->
     <xacro:dermis_base_macro

File: meshes/skin/hybrid/link5_hybrid_front.xacro (robot description, xacro)
@@ -5,5 +5,5 @@
     <!-- Properties -->
     <xacro:property name="use_mesh_file" value="true" />
-    <xacro:property name="mesh_file" value="package://gentact_descriptions/meshes/skin/hybrid/link5_part1_hybrid_dermis.stl" />
+    <xacro:property name="mesh_file" value="package://gentact_descriptions_hybrid/meshes/skin/hybrid/link5_part1_hybrid_dermis.stl" />
     <xacro:property name="mass" value="0.3" /> <!-- [kg] -->
     <xacro:property name="body_width" value="0.3" /> <!-- [m] -->
@@ -12,5 +12,5 @@
     <xacro:property name="sensor_radius" value="0.0" /> <!-- [m] -->
     <!-- Included URDF Files -->
-    <xacro:include filename="$(find gentact_ros_tools)/urdf/skin/self-cap-base.xacro" />
+    <xacro:include filename="$(find gentact_ros_tools_hybrid)/urdf/skin/self-cap-base.xacro" />
     <!-- Instantiate dermis once -->
     <xacro:dermis_base_macro

File: meshes/skin/hybrid/link6_hybrid.xacro (robot description, xacro)
@@ -5,5 +5,5 @@
     <!-- Properties -->
     <xacro:property name="use_mesh_file" value="true" />
-    <xacro:property name="mesh_file" value="package://gentact_descriptions/meshes/skin/hybrid/link6_hybrid_dermis.stl" />
+    <xacro:property name="mesh_file" value="package://gentact_descriptions_hybrid/meshes/skin/hybrid/link6_hybrid_dermis.stl" />
     <xacro:property name="mass" value="0.3" /> <!-- [kg] -->
     <xacro:property name="body_width" value="0.3" /> <!-- [m] -->
@@ -12,5 +12,5 @@
     <xacro:property name="sensor_radius" value="0.0" /> <!-- [m] -->
     <!-- Included URDF Files -->
-    <xacro:include filename="$(find gentact_ros_tools)/urdf/skin/self-cap-base.xacro" />
+    <xacro:include filename="$(find gentact_ros_tools_hybrid)/urdf/skin/self-cap-base.xacro" />
     <!-- Instantiate dermis once -->
     <xacro:dermis_base_macro

File: urdf/calibration/link2.xacro (robot description, xacro)
@@ -2,5 +2,5 @@
 <robot name="calibration_skin" xmlns:xacro="http://ros.org/wiki/xacro">
   <!-- Include the link5 skin macro -->
-  <xacro:include filename="$(find gentact_ros_tools)/urdf/skin/link2_fancy.xacro" />
+  <xacro:include filename="$(find gentact_ros_tools_hybrid)/urdf/skin/link2_fancy.xacro" />
   <!-- Create a base link for the calibration skin -->
   <link name="calibration_base" />

File: urdf/compiled/fr3_hybrid_skin.urdf (robot description, URDF)
Before this commit: robot fr3, 53 links, 52 joints
Links:
- added link link1_sensor_0
- added link link1_sensor_1
- added link link1_sensor_2
- added link link1_sensor_3
- added link link1_sensor_4
- added link link1_sensor_5
- added link link1_sensor_6
- added link link1_skin; visual mesh filename=package://gentact_descriptions_hybrid/meshes/skin/hybrid/li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 scale=0.001 0.001 0.001
- link fr3_hand: geometry collision mesh filename=package://gentact_descriptions_hybrid/meshes/robot_ee/frank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; visual mesh filename=package://gentact_descriptions/meshes/robot_ee/franka_hand_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
- link fr3_link0: geometry collision mesh filename=package://gentact_descriptions_hybrid/meshes/robot_arms/fr3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; visual mesh filename=package://gentact_descriptions_hybrid/meshes/robot_arms/fr3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
- link fr3_link1: geometry collision mesh filename=package://gentact_descriptions_hybrid/meshes/robot_arms/fr3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; visual mesh filename=package://gentact_descriptions_hybrid/meshes/robot_arms/fr3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
- link fr3_link2: geometry collision mesh filename=package://gentact_descriptions_hybrid/meshes/robot_arms/fr3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; visual mesh filename=package://gentact_descriptions_hybrid/meshes/robot_arms/fr3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
- link fr3_link3: geometry collision mesh filename=package://gentact_descriptions_hybrid/meshes/robot_arms/fr3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; visual mesh filename=package://gentact_descriptions_hybrid/meshes/robot_arms/fr3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
- link fr3_link4: geometry collision mesh filename=package://gentact_descriptions_hybrid/meshes/robot_arms/fr3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; visual mesh filename=package://gentact_descriptions_hybrid/meshes/robot_arms/fr3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
- link fr3_link5: geometry collision mesh filename=package://gentact_descriptions_hybrid/meshes/robot_arms/fr3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; visual mesh filename=package://gentact_descriptions_hybrid/meshes/robot_arms/fr3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
- link fr3_link6: geometry collision mesh filename=package://gentact_descriptions_hybrid/meshes/robot_arms/fr3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; visual mesh filename=package://gentact_descriptions_hybrid/meshes/robot_arms/fr3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
- link fr3_link7: geometry collision mesh filename=package://gentact_descriptions_hybrid/meshes/robot_arms/fr3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; visual mesh filename=package://gentact_descriptions_hybrid/meshes/robot_arms/fr3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
- link link2_skin: geometry visual mesh filename=package://gentact_descriptions_hybrid/meshes/skin/hybrid/li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 scale=0.001 0.001 0.001
- link link3_skin: geometry visual mesh filename=package://gentact_descriptions_hybrid/meshes/skin/hybrid/li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 scale=0.001 0.001 0.001
- link link4_skin: geometry visual mesh filename=package://gentact_descriptions_hybrid/meshes/skin/hybrid/li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 scale=0.001 0.001 0.001
- link link5_back_skin: geometry visual mesh filename=package://gentact_descriptions_hybrid/meshes/skin/hybrid/li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 scale=0.001 0.001 0.001
- link link5_front_skin: geometry visual mesh filename=package://gentact_descriptions_hybrid/meshes/skin/hybrid/li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 scale=0.001 0.001 0.001
- link link6_skin: geometry visual mesh filename=package://gentact_descriptions_hybrid/meshes/skin/hybrid/li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 scale=0.001 0.001 0.001
Joints:
- added joint link1_base_joint: type fixed, parent fr3_link1, child link1_skin, origin xyz=0 0 0 rpy=3.14159265359 0 0
- added joint link1_sensor_0_joint: type fixed, parent link1_skin, child link1_sensor_0, origin xyz=0.007 0.136 -0.007 rpy=-1.463 -3.142 -0.106, axis 0.106 0.989 -0.108
- added joint link1_sensor_1_joint: type fixed, parent link1_skin, child link1_sensor_1, origin xyz=-0.024 0.113 0.045 rpy=0.869 -0.000 -2.678, axis -0.341 0.683 0.646
- added joint link1_sensor_2_joint: type fixed, parent link1_skin, child link1_sensor_2, origin xyz=-0.050 0.113 -0.009 rpy=1.630 -0.000 -2.249, axis -0.777 0.627 -0.06
- added joint link1_sensor_3_joint: type fixed, parent link1_skin, child link1_sensor_3, origin xyz=0.052 0.111 -0.004 rpy=1.627 -0.000 2.332, axis 0.723 0.688 -0.056
- added joint link1_sensor_4_joint: type fixed, parent link1_skin, child link1_sensor_4, origin xyz=0.029 0.112 0.042 rpy=0.893 0.000 2.514, axis 0.458 0.631 0.627
- added joint link1_sensor_5_joint: type fixed, parent link1_skin, child link1_sensor_5, origin xyz=0.009 0.064 0.131 rpy=1.466 0.000 2.917, axis 0.222 0.969 0.105
- added joint link1_sensor_6_joint: type fixed, parent link1_skin, child link1_sensor_6, origin xyz=-0.009 0.112 -0.051 rpy=-0.668 -3.142 0.217, axis -0.133 0.605 -0.785
- joint link2_base_joint: origin xyz=0 0 0 rpy=-1.5707 0 0 -> xyz=0 0 0 rpy=1.5707 0 0

File: urdf/robot/fr3_full_skin.xacro (robot description, xacro)
@@ -7,8 +7,8 @@
   <!-- safety_distance: Minimum safety distance in [m] by which the collision volumes are expanded and which is enforced during robot motions -->
   <!-- arm_id: Namespace of the robot arm. Serves to differentiate between arms in case of multiple instances. -->
-  <!-- joint_limits: description of the joint limits that comes from a YAML file. Example definition: ${xacro.load_yaml('$(find gentact_ros_tools)/robots/fr3/joint_limits.yaml')} -->
-  <!-- kinematics: description of the kinematics that comes from a YAML file. Example definition: ${xacro.load_yaml('$(find gentact_ros_tools)/robots/fr3/kinematics.yaml')} -->
-  <!-- inertials: description of the inertials that comes from a YAML file. Example definition: ${xacro.load_yaml('$(find gentact_ros_tools)/robots/fr3/inertials.yaml')} -->
-  <!-- dynamics: description of the dynamics that comes from a YAML file. Example definition: ${xacro.load_yaml('$(find gentact_ros_tools)/robots/fr3/dynamics.yaml')} -->
+  <!-- joint_limits: description of the joint limits that comes from a YAML file. Example definition: ${xacro.load_yaml('$(find gentact_ros_tools_hybrid)/robots/fr3/joint_limits.yaml')} -->
+  <!-- kinematics: description of the kinematics that comes from a YAML file. Example definition: ${xacro.load_yaml('$(find gentact_ros_tools_hybrid)/robots/fr3/kinematics.yaml')} -->
+  <!-- inertials: description of the inertials that comes from a YAML file. Example definition: ${xacro.load_yaml('$(find gentact_ros_tools_hybrid)/robots/fr3/inertials.yaml')} -->
+  <!-- dynamics: description of the dynamics that comes from a YAML file. Example definition: ${xacro.load_yaml('$(find gentact_ros_tools_hybrid)/robots/fr3/dynamics.yaml')} -->
   <!-- Define arguments for skin configurations -->
   <xacro:arg name="link1_skin" default=""/>
@@ -31,10 +31,10 @@
     <visual name="fr3_link0_visual">
       <geometry>
-        <mesh filename="package://gentact_ros_tools/meshes/robot_arms/fr3/visual/link0.dae"/>
+        <mesh filename="package://gentact_ros_tools_hybrid/meshes/robot_arms/fr3/visual/link0.dae"/>
       </geometry>
     </visual>
     <collision name="fr3_link0_collision">
       <geometry>
-        <mesh filename="package://gentact_ros_tools/meshes/robot_arms/fr3/collision/link0.stl"/>
+        <mesh filename="package://gentact_ros_tools_hybrid/meshes/robot_arms/fr3/collision/link0.stl"/>
       </geometry>
     </collision>
@@ -49,10 +49,10 @@
     <visual name="fr3_link1_visual">
       <geometry>
-        <mesh filename="package://gentact_ros_tools/meshes/robot_arms/fr3/visual/link1.dae"/>
+        <mesh filename="package://gentact_ros_tools_hybrid/meshes/robot_arms/fr3/visual/link1.dae"/>
       </geometry>
     </visual>
     <collision name="fr3_link1_collision">
       <geometry>
-        <mesh filename="package://gentact_ros_tools/meshes/robot_arms/fr3/collision/link1.stl"/>
+        <mesh filename="package://gentact_ros_tools_hybrid/meshes/robot_arms/fr3/collision/link1.stl"/>
       </geometry>
     </collision>
@@ -82,10 +82,10 @@
     <visual name="fr3_link2_visual">
       <geometry>
-        <mesh filename="package://gentact_ros_tools/meshes/robot_arms/fr3/visual/link2.dae"/>
+        <mesh filename="package://gentact_ros_tools_hybrid/meshes/robot_arms/fr3/visual/link2.dae"/>
       </geometry>
     </visual>
     <collision name="fr3_link2_collision">
       <geometry>
-        <mesh filename="package://gentact_ros_tools/meshes/robot_arms/fr3/collision/link2.stl"/>
+        <mesh filename="package://gentact_ros_tools_hybrid/meshes/robot_arms/fr3/collision/link2.stl"/>
       </geometry>
     </collision>
@@ -115,10 +115,10 @@
     <visual name="fr3_link3_visual">
       <geometry>
-        <mesh filename="package://gentact_ros_tools/meshes/robot_arms/fr3/visual/link3.dae"/>
+        <mesh filename="package://gentact_ros_tools_hybrid/meshes/robot_arms/fr3/visual/link3.dae"/>
       </geometry>
     </visual>
     <collision name="fr3_link3_collision">
       <geometry>
-        <mesh filename="package://gentact_ros_tools/meshes/robot_arms/fr3/collision/link3.stl"/>
+        <mesh filename="package://gentact_ros_tools_hybrid/meshes/robot_arms/fr3/collision/link3.stl"/>
       </geometry>
     </collision>
@@ -148,10 +148,10 @@
     <visual name="fr3_link4_visual">
       <geometry>
-        <mesh filename="package://gentact_ros_tools/meshes/robot_arms/fr3/visual/link4.dae"/>
+        <mesh filename="package://gentact_ros_tools_hybrid/meshes/robot_arms/fr3/visual/link4.dae"/>
       </geometry>
     </visual>
     <collision name="fr3_link4_collision">
       <geometry>
-        <mesh filename="package://gentact_ros_tools/meshes/robot_arms/fr3/collision/link4.stl"/>
+        <mesh filename="package://gentact_ros_tools_hybrid/meshes/robot_arms/fr3/collision/link4.stl"/>
       </geometry>
     </collision>
@@ -181,10 +181,10 @@
     <visual name="fr3_link5_visual">
       <geometry>
-        <mesh filename="package://gentact_ros_tools/meshes/robot_arms/fr3/visual/link5.dae"/>
+        <mesh filename="package://gentact_ros_tools_hybrid/meshes/robot_arms/fr3/visual/link5.dae"/>
       </geometry>
     </visual>
     <collision name="fr3_link5_collision">
       <geometry>
-        <mesh filename="package://gentact_ros_tools/meshes/robot_arms/fr3/collision/link5.stl"/>
+        <mesh filename="package://gentact_ros_tools_hybrid/meshes/robot_arms/fr3/collision/link5.stl"/>
       </geometry>
     </collision>
@@ -220,10 +220,10 @@
     <visual name="fr3_link6_visual">
       <geometry>
-        <mesh filename="package://gentact_ros_tools/meshes/robot_arms/fr3/visual/link6.dae"/>
+        <mesh filename="package://gentact_ros_tools_hybrid/meshes/robot_arms/fr3/visual/link6.dae"/>
       </geometry>
     </visual>
     <collision name="fr3_link6_collision">
       <geometry>
-        <mesh filename="package://gentact_ros_tools/meshes/robot_arms/fr3/collision/link6.stl"/>
+        <mesh filename="package://gentact_ros_tools_hybrid/meshes/robot_arms/fr3/collision/link6.stl"/>
       </geometry>
     </collision>
@@ -253,10 +253,10 @@
     <visual name="fr3_link7_visual">
       <geometry>
-        <mesh filename="package://gentact_ros_tools/meshes/robot_arms/fr3/visual/link7.dae"/>
+        <mesh filename="package://gentact_ros_tools_hybrid/meshes/robot_arms/fr3/visual/link7.dae"/>
       </geometry>
     </visual>
     <collision name="fr3_link7_collision">
       <geometry>
-        <mesh filename="package://gentact_ros_tools/meshes/robot_arms/fr3/collision/link7.stl"/>
+        <mesh filename="package://gentact_ros_tools_hybrid/meshes/robot_arms/fr3/collision/link7.stl"/>
       </geometry>
     </collision>
