Commit message: add link2 correct orientation

File: urdf/skin/hybrid/link1_hybrid.xacro (robot description, xacro)
@@ -2,8 +2,8 @@
 <robot xmlns:xacro="http://ros.org/wiki/xacro">
   <!-- Macro definition for link2 skin -->
-  <xacro:macro name="link2_skin" params="parent namespace">
+  <xacro:macro name="link1_skin" params="parent namespace">
     <!-- Properties -->
     <xacro:property name="use_mesh_file" value="true" />
-    <xacro:property name="mesh_file" value="package://gentact_descriptions_hybrid/meshes/skin/hybrid/link2_hybrid_dermis.stl" />
+    <xacro:property name="mesh_file" value="package://gentact_ros_tools_hybrid/meshes/skin/hybrid/link1_hybrid_dermis.stl" />
     <xacro:property name="mass" value="0.3" /> <!-- [kg] -->
     <xacro:property name="body_width" value="0.3" /> <!-- [m] -->
@@ -12,5 +12,5 @@
     <xacro:property name="sensor_radius" value="0.0" /> <!-- [m] -->
     <!-- Included URDF Files -->
-    <xacro:include filename="$(find gentact_descriptions_hybrid)/robots/common/skin_unit_base.xacro" />
+    <xacro:include filename="$(find gentact_ros_tools_hybrid)/urdf/skin/self-cap-base.xacro" />
     <!-- Instantiate dermis once -->
     <xacro:dermis_base_macro
@@ -22,35 +22,34 @@
       use_mesh_file="${use_mesh_file}"
       mesh_file="${mesh_file}">
-      <origin xyz="0 0 0" rpy="-1.5707 0 0" />
+        <origin xyz="0 0 0" rpy="-3.14159265359 0 0" />
     </xacro:dermis_base_macro>
-    <!-- Instantiate sensors -->
     <xacro:self_cap_sensor robot_namespace="${namespace}" parent="${namespace}_skin" sensor_number="0"
+      sensor_radius="${sensor_radius}" sensor_length="${sensor_length}" normal_x="0.106" normal_y="0.989" normal_z="-0.108">
+      <origin xyz="0.007 0.136 -0.007" rpy="-1.463 -3.142 -0.106" />
+    </xacro:self_cap_sensor>
+    <xacro:self_cap_sensor robot_namespace="${namespace}" parent="${namespace}_skin" sensor_number="1"
+      sensor_radius="${sensor_radius}" sensor_length="${sensor_length}" normal_x="-0.341" normal_y="0.683" normal_z="0.646">
+      <origin xyz="-0.024 0.113 0.045" rpy="0.869 -0.000 -2.678" />
+    </xacro:self_cap_sensor>
+    <xacro:self_cap_sensor robot_namespace="${namespace}" parent="${namespace}_skin" sensor_number="2"
+      sensor_radius="${sensor_radius}" sensor_length="${sensor_length}" normal_x="-0.777" normal_y="0.627" normal_z="-0.060">
+      <origin xyz="-0.050 0.113 -0.009" rpy="1.630 -0.000 -2.249" />
+    </xacro:self_cap_sensor>
+    <xacro:self_cap_sensor robot_namespace="${namespace}" parent="${namespace}_skin" sensor_number="3"
       sensor_radius="${sensor_radius}" sensor_length="${sensor_length}" normal_x="0.723" normal_y="0.688" normal_z="-0.056">
       <origin xyz="0.052 0.111 -0.004" rpy="1.627 -0.000 2.332" />
     </xacro:self_cap_sensor>
-    <xacro:self_cap_sensor robot_namespace="${namespace}" parent="${namespace}_skin" sensor_number="1"
+    <xacro:self_cap_sensor robot_namespace="${namespace}" parent="${namespace}_skin" sensor_number="4"
       sensor_radius="${sensor_radius}" sensor_length="${sensor_length}" normal_x="0.458" normal_y="0.631" normal_z="0.627">
       <origin xyz="0.029 0.112 0.042" rpy="0.893 0.000 2.514" />
     </xacro:self_cap_sensor>
-    <xacro:self_cap_sensor robot_namespace="${namespace}" parent="${namespace}_skin" sensor_number="2"
-      sensor_radius="${sensor_radius}" sensor_length="${sensor_length}" normal_x="0.106" normal_y="0.989" normal_z="-0.108">
-      <origin xyz="0.007 0.136 -0.007" rpy="-1.463 -3.142 -0.106" />
-    </xacro:self_cap_sensor>
-    <xacro:self_cap_sensor robot_namespace="${namespace}" parent="${namespace}_skin" sensor_number="3"
+    <xacro:self_cap_sensor robot_namespace="${namespace}" parent="${namespace}_skin" sensor_number="5"
       sensor_radius="${sensor_radius}" sensor_length="${sensor_length}" normal_x="0.222" normal_y="0.969" normal_z="0.105">
       <origin xyz="0.009 0.064 0.131" rpy="1.466 0.000 2.917" />
     </xacro:self_cap_sensor>
-    <xacro:self_cap_sensor robot_namespace="${namespace}" parent="${namespace}_skin" sensor_number="4"
+    <xacro:self_cap_sensor robot_namespace="${namespace}" parent="${namespace}_skin" sensor_number="6"
       sensor_radius="${sensor_radius}" sensor_length="${sensor_length}" normal_x="-0.133" normal_y="0.605" normal_z="-0.785">
       <origin xyz="-0.009 0.112 -0.051" rpy="-0.668 -3.142 0.217" />
     </xacro:self_cap_sensor>
-    <xacro:self_cap_sensor robot_namespace="${namespace}" parent="${namespace}_skin" sensor_number="5"
-      sensor_radius="${sensor_radius}" sensor_length="${sensor_length}" normal_x="-0.341" normal_y="0.683" normal_z="0.646">
-      <origin xyz="-0.024 0.113 0.045" rpy="0.869 -0.000 -2.678" />
-    </xacro:self_cap_sensor>
-    <xacro:self_cap_sensor robot_namespace="${namespace}" parent="${namespace}_skin" sensor_number="6"
-      sensor_radius="${sensor_radius}" sensor_length="${sensor_length}" normal_x="-0.777" normal_y="0.627" normal_z="-0.060">
-      <origin xyz="-0.050 0.113 -0.009" rpy="1.630 -0.000 -2.249" />
-    </xacro:self_cap_sensor>
   </xacro:macro>
      </robot>

File: urdf/skin/hybrid/link2_hybrid.xacro (robot description, xacro)
@@ -5,5 +5,5 @@
     <!-- Properties -->
     <xacro:property name="use_mesh_file" value="true" />
-    <xacro:property name="mesh_file" value="package://gentact_ros_tools/meshes/skin/hybrid/link2_hybrid_dermis.stl" />
+    <xacro:property name="mesh_file" value="package://gentact_ros_tools_hybrid/meshes/skin/hybrid/link2_hybrid_dermis.stl" />
     <xacro:property name="mass" value="0.3" /> <!-- [kg] -->
     <xacro:property name="body_width" value="0.3" /> <!-- [m] -->
@@ -12,5 +12,5 @@
     <xacro:property name="sensor_radius" value="0.0" /> <!-- [m] -->
     <!-- Included URDF Files -->
-    <xacro:include filename="$(find gentact_ros_tools)/urdf/skin/self-cap-base.xacro" />
+    <xacro:include filename="$(find gentact_ros_tools_hybrid)/urdf/skin/self-cap-base.xacro" />
     <!-- Instantiate dermis once -->
     <xacro:dermis_base_macro
@@ -22,5 +22,5 @@
       use_mesh_file="${use_mesh_file}"
       mesh_file="${mesh_file}">
-      <origin xyz="0 0 0" rpy="-1.5707 0 0" />
+      <origin xyz="0 0 0" rpy="1.5707 0 0" />
     </xacro:dermis_base_macro>
     <!-- Instantiate sensors -->

File: urdf/skin/hybrid/link3_hybrid.xacro (robot description, xacro)
@@ -5,5 +5,5 @@
     <!-- Properties -->
     <xacro:property name="use_mesh_file" value="true" />
-    <xacro:property name="mesh_file" value="package://gentact_ros_tools/meshes/skin/hybrid/link3_hybrid_dermis.stl" />
+    <xacro:property name="mesh_file" value="package://gentact_ros_tools_hybrid/meshes/skin/hybrid/link3_hybrid_dermis.stl" />
     <xacro:property name="mass" value="0.3" /> <!-- [kg] -->
     <xacro:property name="body_width" value="0.3" /> <!-- [m] -->
@@ -12,5 +12,5 @@
     <xacro:property name="sensor_radius" value="0.0" /> <!-- [m] -->
     <!-- Included URDF Files -->
-    <xacro:include filename="$(find gentact_ros_tools)/urdf/skin/self-cap-base.xacro" />
+    <xacro:include filename="$(find gentact_ros_tools_hybrid)/urdf/skin/self-cap-base.xacro" />
     <!-- Instantiate dermis once -->
     <xacro:dermis_base_macro

File: urdf/skin/hybrid/link4_hybrid.xacro (robot description, xacro)
@@ -5,5 +5,5 @@
     <!-- Properties -->
     <xacro:property name="use_mesh_file" value="true" />
-    <xacro:property name="mesh_file" value="package://gentact_ros_tools/meshes/skin/hybrid/link4_hybrid_dermis.stl" />
+    <xacro:property name="mesh_file" value="package://gentact_ros_tools_hybrid/meshes/skin/hybrid/link4_hybrid_dermis.stl" />
     <xacro:property name="mass" value="0.3" /> <!-- [kg] -->
     <xacro:property name="body_width" value="0.3" /> <!-- [m] -->
@@ -12,5 +12,5 @@
     <xacro:property name="sensor_radius" value="0.0" /> <!-- [m] -->
     <!-- Included URDF Files -->
-    <xacro:include filename="$(find gentact_ros_tools)/urdf/skin/self-cap-base.xacro" />
+    <xacro:include filename="$(find gentact_ros_tools_hybrid)/urdf/skin/self-cap-base.xacro" />
     <!-- Instantiate dermis once -->
     <xacro:dermis_base_macro

File: urdf/skin/hybrid/link5_hybrid_back.xacro (robot description, xacro)
@@ -5,5 +5,5 @@
     <!-- Properties -->
     <xacro:property name="use_mesh_file" value="true" />
-    <xacro:property name="mesh_file" value="package://gentact_ros_tools/meshes/skin/hybrid/link5_part2_hybrid_dermis.stl" />
+    <xacro:property name="mesh_file" value="package://gentact_ros_tools_hybrid/meshes/skin/hybrid/link5_part2_hybrid_dermis.stl" />
     <xacro:property name="mass" value="0.3" /> <!-- [kg] -->
     <xacro:property name="body_width" value="0.3" /> <!-- [m] -->
@@ -12,5 +12,5 @@
     <xacro:property name="sensor_radius" value="0.0" /> <!-- [m] -->
     <!-- Included URDF Files -->
-    <xacro:include filename="$(find gentact_ros_tools)/urdf/skin/self-cap-base.xacro" />
+    <xacro:include filename="$(find gentact_ros_tools_hybrid)/urdf/skin/self-cap-base.xacro" />
     <!-- Instantiate dermis once -->
     <xacro:dermis_base_macro

File: urdf/skin/hybrid/link5_hybrid_front.xacro (robot description, xacro)
@@ -5,5 +5,5 @@
     <!-- Properties -->
     <xacro:property name="use_mesh_file" value="true" />
-    <xacro:property name="mesh_file" value="package://gentact_ros_tools/meshes/skin/hybrid/link5_part1_hybrid_dermis.stl" />
+    <xacro:property name="mesh_file" value="package://gentact_ros_tools_hybrid/meshes/skin/hybrid/link5_part1_hybrid_dermis.stl" />
     <xacro:property name="mass" value="0.3" /> <!-- [kg] -->
     <xacro:property name="body_width" value="0.3" /> <!-- [m] -->
@@ -12,5 +12,5 @@
     <xacro:property name="sensor_radius" value="0.0" /> <!-- [m] -->
     <!-- Included URDF Files -->
-    <xacro:include filename="$(find gentact_ros_tools)/urdf/skin/self-cap-base.xacro" />
+    <xacro:include filename="$(find gentact_ros_tools_hybrid)/urdf/skin/self-cap-base.xacro" />
     <!-- Instantiate dermis once -->
     <xacro:dermis_base_macro

File: urdf/skin/hybrid/link6_hybrid.xacro (robot description, xacro)
@@ -5,5 +5,5 @@
     <!-- Properties -->
     <xacro:property name="use_mesh_file" value="true" />
-    <xacro:property name="mesh_file" value="package://gentact_ros_tools/meshes/skin/hybrid/link6_hybrid_dermis.stl" />
+    <xacro:property name="mesh_file" value="package://gentact_ros_tools_hybrid/meshes/skin/hybrid/link6_hybrid_dermis.stl" />
     <xacro:property name="mass" value="0.3" /> <!-- [kg] -->
     <xacro:property name="body_width" value="0.3" /> <!-- [m] -->
@@ -12,5 +12,5 @@
     <xacro:property name="sensor_radius" value="0.0" /> <!-- [m] -->
     <!-- Included URDF Files -->
-    <xacro:include filename="$(find gentact_ros_tools)/urdf/skin/self-cap-base.xacro" />
+    <xacro:include filename="$(find gentact_ros_tools_hybrid)/urdf/skin/self-cap-base.xacro" />
     <!-- Instantiate dermis once -->
     <xacro:dermis_base_macro
