Commit message: added go1 urdf

File: urdf/compiled/h1_2/h1_2_handless_tof.urdf (robot description, URDF)
Before this commit: robot h1_2, 114 links, 113 joints
Links:
- link left_ankle_pitch_link: geometry visual mesh filename=package://gentact_ros_tools_hybrid/meshes/h1_2/left_ankle_p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
- link left_ankle_roll_link: geometry collision mesh filename=package://gentact_ros_tools_hybrid/meshes/h1_2/left_ankle_r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; visual mesh filename=package://gentact_ros_tools_hybrid/meshes/h1_2/left_ankle_r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
- link left_elbow_link: geometry collision mesh filename=package://gentact_ros_tools_hybrid/meshes/h1_2/left_elbow_l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; visual mesh filename=package://gentact_ros_tools_hybrid/meshes/h1_2/left_elbow_l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
- link left_hip_pitch_link: geometry collision mesh filename=package://gentact_ros_tools_hybrid/meshes/h1_2/left_hip_pit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; visual mesh filename=package://gentact_ros_tools_hybrid/meshes/h1_2/left_hip_pit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
- link left_hip_roll_link: geometry collision mesh filename=package://gentact_ros_tools_hybrid/meshes/h1_2/left_hip_rol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; visual mesh filename=package://gentact_ros_tools_hybrid/meshes/h1_2/left_hip_rol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
- link left_hip_yaw_link: geometry visual mesh filename=package://gentact_ros_tools_hybrid/meshes/h1_2/left_hip_yaw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
- link left_knee_link: geometry collision cylinder length=0.2 radius=0.04; visual mesh filename=package://gentact_ros_tools_hybrid/meshes/h1_2/left_knee_li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
- link left_shoulder_pitch_link: geometry collision mesh filename=package://gentact_ros_tools_hybrid/meshes/h1_2/left_shoulde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; visual mesh filename=package://gentact_ros_tools_hybrid/meshes/h1_2/left_shoulde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
- link left_shoulder_roll_link: geometry collision mesh filename=package://gentact_ros_tools_hybrid/meshes/h1_2/left_shoulde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; visual mesh filename=package://gentact_ros_tools_hybrid/meshes/h1_2/left_shoulde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
- link left_shoulder_yaw_link: geometry collision mesh filename=package://gentact_ros_tools_hybrid/meshes/h1_2/left_shoulde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; visual mesh filename=package://gentact_ros_tools_hybrid/meshes/h1_2/left_shoulde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
- link left_wrist_pitch_link: geometry collision mesh filename=package://gentact_ros_tools_hybrid/meshes/h1_2/left_wrist_p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; visual mesh filename=package://gentact_ros_tools_hybrid/meshes/h1_2/left_wrist_p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
- link left_wrist_roll_link: geometry collision mesh filename=package://gentact_ros_tools_hybrid/meshes/h1_2/left_wrist_r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; visual mesh filename=package://gentact_ros_tools_hybrid/meshes/h1_2/left_wrist_r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
- link left_wrist_yaw_link: geometry visual mesh filename=package://gentact_ros_tools_hybrid/meshes/h1_2/wrist_yaw_li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
- link logo_link: geometry visual mesh filename=package://gentact_ros_tools_hybrid/meshes/h1_2/logo_link.STL
- link pelvis: geometry collision mesh filename=package://gentact_ros_tools_hybrid/meshes/h1_2/pelvis.STL; visual mesh filename=package://gentact_ros_tools_hybrid/meshes/h1_2/pelvis.STL
- link right_ankle_pitch_link: geometry visual mesh filename=package://gentact_ros_tools_hybrid/meshes/h1_2/right_ankle_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
- link right_ankle_roll_link: geometry collision mesh filename=package://gentact_ros_tools_hybrid/meshes/h1_2/right_ankle_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; visual mesh filename=package://gentact_ros_tools_hybrid/meshes/h1_2/right_ankle_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
- link right_elbow_link: geometry collision mesh filename=package://gentact_ros_tools_hybrid/meshes/h1_2/right_elbow_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; visual mesh filename=package://gentact_ros_tools_hybrid/meshes/h1_2/right_elbow_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
- link right_hip_pitch_link: geometry collision mesh filename=package://gentact_ros_tools_hybrid/meshes/h1_2/right_hip_pi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; visual mesh filename=package://gentact_ros_tools_hybrid/meshes/h1_2/right_hip_pi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
- link right_hip_roll_link: geometry collision mesh filename=package://gentact_ros_tools_hybrid/meshes/h1_2/right_hip_ro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; visual mesh filename=package://gentact_ros_tools_hybrid/meshes/h1_2/right_hip_ro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
- link right_hip_yaw_link: geometry visual mesh filename=package://gentact_ros_tools_hybrid/meshes/h1_2/right_hip_ya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
- link right_knee_link: geometry collision cylinder length=0.2 radius=0.04; visual mesh filename=package://gentact_ros_tools_hybrid/meshes/h1_2/right_knee_l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
- link right_shoulder_pitch_link: geometry collision mesh filename=package://gentact_ros_tools_hybrid/meshes/h1_2/right_should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; visual mesh filename=package://gentact_ros_tools_hybrid/meshes/h1_2/right_should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
- link right_shoulder_roll_link: geometry collision mesh filename=package://gentact_ros_tools_hybrid/meshes/h1_2/right_should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; visual mesh filename=package://gentact_ros_tools_hybrid/meshes/h1_2/right_should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
- link right_shoulder_yaw_link: geometry collision mesh filename=package://gentact_ros_tools_hybrid/meshes/h1_2/right_should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; visual mesh filename=package://gentact_ros_tools_hybrid/meshes/h1_2/right_should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
- link right_wrist_pitch_link: geometry collision mesh filename=package://gentact_ros_tools_hybrid/meshes/h1_2/right_wrist_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; visual mesh filename=package://gentact_ros_tools_hybrid/meshes/h1_2/right_wrist_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
- link right_wrist_roll_link: geometry collision mesh filename=package://gentact_ros_tools_hybrid/meshes/h1_2/right_wrist_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; visual mesh filename=package://gentact_ros_tools_hybrid/meshes/h1_2/right_wrist_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
- link right_wrist_yaw_link: geometry visual mesh filename=package://gentact_ros_tools_hybrid/meshes/h1_2/wrist_yaw_li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
- link torso_link: geometry collision mesh filename=package://gentact_ros_tools_hybrid/meshes/h1_2/torso_link.S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; visual mesh filename=package://gentact_ros_tools_hybrid/meshes/h1_2/torso_link.S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
