Commit message: fix urdf (thighcap poses correct)

File: urdf/compiled/go-1/go1_tof_skins.urdf (robot description, URDF)
Before this commit: robot go1, 72 links, 71 joints
Links:
- added link trunk_head_sensor_3
- added link trunk_head_sensor_4
- link left_thighcap_skin: geometry visual mesh filename=package://gentact_ros_tools_hybrid/meshes/go-1/skin/thigh/l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 scale=1 1 1
- link right_thighcap_skin: geometry visual mesh filename=package://gentact_ros_tools_hybrid/meshes/go-1/skin/thigh/r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 scale=1 1 1
Joints:
- added joint trunk_head_sensor_3_joint: type fixed, parent trunk_head_skin, child trunk_head_sensor_3, origin xyz=-0.06460931897163391 -0.27623823285102844 0.0038362115155905485 rpy=1.494691252708435 -0.024021487683057785 -0.30515751242637634, axis 1.494691252708435 -0.024021487683057785 -0.30515751242637634
- added joint trunk_head_sensor_4_joint: type fixed, parent trunk_head_skin, child trunk_head_sensor_4, origin xyz=0.06688925623893738 -0.2754700481891632 0.00686574075371027 rpy=1.4878184795379639 0.02471890300512314 0.2888708710670471, axis 1.4878184795379639 0.02471890300512314 0.2888708710670471
- joint left_thighcap_sensor_0_joint: origin xyz=0.006742224097251892 0.014293902553617954 0.029223144054412842 rpy=-1.2252006530761719 -0.005685813259333372 0.0157905425876379 -> xyz=0.0010693295625969768 -0.006162808742374182 0.046794019639492035 rpy=-1.2252006530761719 -0.005685813259333372 0.0157905425876379
- joint left_thighcap_sensor_1_joint: origin xyz=-0.037725191563367844 -0.0013956413604319096 0.008954118005931377 rpy=-1.3508657217025757 -0.3039449453353882 0.9292620420455933 -> xyz=-0.0425979383289814 -0.008709190413355827 0.021811174228787422 rpy=-1.3508657217025757 -0.3039449453353882 0.9292620420455933
- joint left_thighcap_sensor_2_joint: origin xyz=0.0007210002513602376 0.013414165005087852 -0.016765158623456955 rpy=-2.012596607208252 0.012588809244334698 0.026608869433403015 -> xyz=-0.004939308390021324 0.01649658940732479 0.0077791460789740086 rpy=-2.012596607208252 0.012588809244334698 0.026608869433403015
- joint right_thighcap_sensor_0_joint: origin xyz=0.006742224097251892 -0.014293902553617954 0.029223144054412842 rpy=-1.2252006530761719 -0.005685813259333372 0.0157905425876379 -> xyz=0.0010693295625969768 0.007912559434771538 0.046794019639492035 rpy=-1.2252006530761719 -0.005685813259333372 0.0157905425876379
- joint right_thighcap_sensor_1_joint: origin xyz=-0.037725191563367844 0.0013956413604319096 0.008954118005931377 rpy=-1.3508657217025757 -0.3039449453353882 0.9292620420455933 -> xyz=-0.0425979383289814 0.009698150679469109 0.021811174228787422 rpy=-1.3508657217025757 -0.3039449453353882 0.9292620420455933
- joint right_thighcap_sensor_2_joint: origin xyz=0.0007210002513602376 -0.013414165005087852 -0.016765158623456955 rpy=-2.012596607208252 0.012588809244334698 0.026608869433403015 -> xyz=-0.004939308390021324 -0.01481604017317295 0.0077791460789740086 rpy=-2.012596607208252 0.012588809244334698 0.026608869433403015
- joint trunk_head_base_joint: origin xyz=0 0 0 rpy=0 0 0 -> xyz=0.275155 0.001302 0.010202 rpy=0 0 1.570796
- joint trunk_head_sensor_0_joint: axis -1.5642733573913574 -0.0002883475972339511 0.0441758893430233 -> 1.2075234651565552 -0.007908201776444912 -0.020799949765205383; origin xyz=-0.020546915009617805 0.016203830018639565 -0.13735900819301605 rpy=-1.5642733573913574 -0.0002883475972339511 0.0441758893430233 -> xyz=0.00025236696819774806 -0.2968325912952423 0.04981664940714836 rpy=1.2075234651565552 -0.007908201776444912 -0.020799949765205383
- joint trunk_head_sensor_1_joint: axis -1.6060417890548706 -0.0003777451638597995 -0.010712702758610249 -> 1.1489475965499878 -0.39848679304122925 -0.7129077315330505; origin xyz=-0.00846764538437128 0.016201069578528404 -0.046428292989730835 rpy=-1.6060417890548706 -0.0003777451638597995 -0.010712702758610249 -> xyz=-0.03770412877202034 -0.2818562388420105 0.051483239978551865 rpy=1.1489475965499878 -0.39848679304122925 -0.7129077315330505
- joint trunk_head_sensor_2_joint: axis 1.6190142631530762 -0.024614643305540085 -1.5761873722076416 -> 1.1440706253051758 0.4009367823600769 0.7093470692634583; origin xyz=-0.0421280711889267 0.000184581644134596 -0.10028665512800217 rpy=-2.077631950378418 1.4713668823242188 1.0618557929992676 -> xyz=0.03843432292342186 -0.28169137239456177 0.05167349427938461 rpy=1.1440706253051758 0.4009367823600769 0.7093470692634583

Commit message: fix head sensor poses

File: urdf/compiled/go-1/go1_tof_skins.urdf (robot description, URDF)
Before this commit: robot go1, 74 links, 73 joints
Joints:
- joint trunk_head_base_joint: origin xyz=0.275155 0.001302 0.010202 rpy=0 0 1.570796 -> xyz=0 0 0 rpy=0 0 0
- joint trunk_head_sensor_0_joint: origin xyz=0.00025236696819774806 -0.2968325912952423 0.04981664940714836 rpy=1.2075234651565552 -0.007908201776444912 -0.020799949765205383 -> xyz=0.29396241903305054 -0.0024843034334480762 0.04981664940714836 rpy=1.2075234651565552 -0.007908201776444912 -0.020799949765205383
- joint trunk_head_sensor_1_joint: origin xyz=-0.03770412877202034 -0.2818562388420105 0.051483239978551865 rpy=1.1489475965499878 -0.39848679304122925 -0.7129077315330505 -> xyz=0.2779468894004822 -0.03731217980384827 0.051483239978551865 rpy=1.1489475965499878 -0.39848679304122925 -0.7129077315330505
- joint trunk_head_sensor_2_joint: origin xyz=0.03843432292342186 -0.28169137239456177 0.05167349427938461 rpy=1.1440706253051758 0.4009367823600769 0.7093470692634583 -> xyz=0.28208127617836 0.03453124314546585 0.05167349427938461 rpy=1.1440706253051758 0.4009367823600769 0.7093470692634583
- joint trunk_head_sensor_3_joint: origin xyz=-0.06460931897163391 -0.27623823285102844 0.0038362115155905485 rpy=1.494691252708435 -0.024021487683057785 -0.30515751242637634 -> xyz=0.27248281240463257 -0.06655683368444443 0.0038362115155905485 rpy=1.494691252708435 -0.024021487683057785 -0.30515751242637634
- joint trunk_head_sensor_4_joint: origin xyz=0.06688925623893738 -0.2754700481891632 0.00686574075371027 rpy=1.4878184795379639 0.02471890300512314 0.2888708710670471 -> xyz=0.27346357703208923 0.06316765397787094 0.00686574075371027 rpy=1.4878184795379639 0.02471890300512314 0.2888708710670471
